File: MR1/MR1.kicad_sch (KiCad schematic)
At the start: 86 parts, among them J1 Conn_Coaxial, J2 Conn_Coaxial, J22 B4B_PH, J23 Jumper_1, J3 USB_C_Receptacle_USB2.0, J36 Conn_ARM_JTAG_SWD_10, J4 Conn_Coaxial, J5 USB B receptical vertical, Q4 DMG2301L, Q5 DMG2301L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

Commit message: Signed-off-by: lokimetasmith <lokimail@gmail.com>
Parts:
- removed C49: 0.1u, Capacitor_SMD:C_0603_1608Metric, symbol Device:C_Small
- removed D4: MBR0540, Diode_SMD:D_SOD-123, symbol Diode:MBR0540
- removed J5: USB B receptical vertical, Connector_USB:USB_B_TE_5787834_Vertical, symbol Connector:USB_B
- removed JP1: ID_WP, Jumper:SolderJumper-2_P1.3mm_Open_TrianglePad1.0x1.5mm, symbol Jumper:SolderJumper_2_Open
- removed Q4, Q5: DMG2301L, Package_TO_SOT_SMD:SOT-23, symbol Transistor_FET:DMG2301L
- removed R132: 27, Resistor_SMD:R_0402_1005Metric, symbol Device:R_Small_US
- removed R18: 100K, Resistor_SMD:R_0402_1005Metric, symbol temp-sensor-rescue:R_Small_US-Device-temp-sensor-rescue
- removed TP1: TestPoint, TestPoint:TestPoint_Pad_D1.0mm, symbol Connector:TestPoint
- removed U6: CAT24C512, Package_SO:SOIC-8_3.9x4.9mm_P1.27mm, symbol Memory_EEPROM:CAT24C256
- added C13, C14, C15, C18: 4.7u, Capacitor_SMD:C_0805_2012Metric, symbol temp-sensor-rescue:C_Small-Device-temp-sensor-rescue
- added C16: 10u, Capacitor_SMD:C_1206_3216Metric, symbol temp-sensor-rescue:C_Small-Device-temp-sensor-rescue
- added J5, J6: Conn_01x05_Socket, symbol Connector:Conn_01x05_Socket
- added JP2: Jumper_2_Bridged, symbol Jumper:Jumper_2_Bridged
- added R18, R23, R24, R25, R26: 10k 1%, Resistor_SMD:R_0402_1005Metric, symbol Device:R_Small_US
- added R19, R20, R21, R22: 5k, Resistor_SMD:R_0805_2012Metric, symbol Device:R
Connections:
- net -5V is gone; now on net VSSA: C3.1, C5.1, U3.4 (V-)
- net VCC_SW_P is gone; now on net VBUS: C10.1, C17.1
- net ANA_0: no longer U8.7 (IO3)
- net ANA_1: no longer U8.6 (IO2)
- net ANA_2: no longer U8.5 (IO1)
- net ANA_3: no longer U8.8 (IO4)
- net GUARD: now also JP2.1 (A); no longer C6.1, R4.1, R6.1, U2.1 (+)
- net SENSE_En: no longer R43.2
- net VBUS: now also D82.1 (K), U1.3 (VIN), C16.1, R23.1
- net Signal: now reaches J2.1 (In), R3.1, U3.6
- net Signal: now also J5.1 (Pin_1), J6.1 (Pin_1)
- net at U4.1 (IN), U4.2 (IN): now also U1.11 (OUT+), C15.2, R24.2
- net at U4.10 (OUT): now also R19.2
- net GNDA: now reaches U4.11 (GND), U4.8 (GND)
- net GNDA: now also U1.13 (PAD), U1.4 (GND), U5.9 (GND), C14.2, C15.1, C16.2, C18.2, J5.3 (Pin_3), J6.3 (Pin_3), R25.1, R26.2
- net at U4.9 (OUTS): now also R19.1, R20.2
- net at U5.1 (IN), U5.13 (IN), U5.2 (IN): now also C14.1, R18.1
- net at U5.10 (OUTS): now also R21.1, R22.2
- net at U5.11 (OUT), U5.12 (OUT): now also R21.2
- net at U1.1 (PGOOD): now also R23.2
- net at U1.10 (C+): now also C13.1
- net at U1.2 (FB+): now also R24.1, R25.2
- net at U1.5 (CP): now also C18.1
- net at U1.7 (FB-): now also R18.2, R26.1
- net at U1.9 (C-): now also C13.2
- net +2.5V renamed VDDA
- net VDDA: now also C2.1, C4.1, J5.2 (Pin_2), J6.2 (Pin_2)
- removed net +5V: C2.1, C4.1, U3.7 (V+)
- net -2.5V renamed VSSA
- net VSSA: now also U3.7 (V+), J5.5 (Pin_5), J6.5 (Pin_5)
- net ETH_CSn renamed GPIO34
- net ETH_En renamed GPIO39
- net GPIO39: no longer J36.4 (SWCLK/TCK)
- net ETH_MISO renamed GPIO37
- net ETH_MOSI renamed GPIO36
- net ETH_SCLK renamed GPIO35
- net Fan_1_Tach renamed GPIO6
- net INTn renamed GPIO21
- net In_0: no longer names the net of R143.1
- net In_1 renamed GPIO8
- net SCL renamed GPIO26
- net SDA renamed GPIO33
- net SD_CSn renamed GPIO41
- net GPIO41: no longer J36.8 (NC/TDI)
- net SSR_CTL1 renamed GPIO10
- net TC_En: no longer names the net of R130.2
- net TC_MUX_A renamed GPIO40
- net GPIO40: no longer J36.6 (SWO/TDO)
- net TC_MUX_B renamed GPIO45
- net TC_MUX_C renamed GPIO46
- net TC_SCK renamed GPIO42
- net GPIO42: no longer J36.2 (SWDIO/TMS)
- net TC_SO renamed GPIO48
- new net GPIO1: U8.5 (IO1)
- new net GPIO2: U8.6 (IO2)
- new net GPIO3: U8.7 (IO3)
- new net GPIO4: U8.8 (IO4)
- new net JTAG_TCK: J36.4 (SWCLK/TCK)
- new net JTAG_TDI: J36.8 (NC/TDI)
- new net JTAG_TDO: J36.6 (SWO/TDO)
- new net JTAG_TMS: J36.2 (SWDIO/TMS)
- new net Vbias: C6.1, J5.4 (Pin_4), J6.4 (Pin_4), JP2.2 (B), R4.1, R6.1, U2.1 (+)
- no-connect marks 5 -> 2
Other:
- note added: "+VOUT = 1.2 V × (R1 + R2) / R2 -VOUT = -1.22 V × (R3 + R4) / R4"
- note added: "PTFE (ZYF255DA): Dk .approx 2.55"
- note removed: "PSU_MISO"
- note removed: "PSU_MOSI"
- note removed: "USB C jtag, debug connector, can optionally provide Power during programming"
- note removed: "Vcc Read-Only GND R/W Enabled"
- moved on the sheet: C1, C10, C17, C2, C3, C4, C5, C6, D82, J1, J2, J3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

Commit message: Signed-off-by: lokimetasmith <lokimail@gmail.com>
Parts:
- added J7: DIN-5_180degree, symbol Connector:DIN-5_180degree
- added NT2: NetTie_2, NetTie:NetTie-2_SMD_Pad0.5mm, symbol Device:NetTie_2
- added U6: MCP3301, symbol Analog_ADC:MCP3301
Connections:
- net GND: now also NT2.2; no longer C2.2, C3.2, C4.2, C5.2, C6.2, J1.2 (Ext), J2.2 (Ext), J4.2 (Ext), R5.2
- net GNDA: now also C2.2, C3.2, C4.2, C5.2, C6.2, J1.2 (Ext), J2.2 (Ext), J4.2 (Ext), R20.1, R22.1, R5.2, NT2.1
- net VDDA: now also R19.1, R20.2, U4.9 (OUTS)
- net VSSA: now also R21.1, R22.2, U5.10 (OUTS)
Other:
- note added: "LTC6268"
- note added: "MCP33131"
- note added: "TODO: update ADC with correct library part and footprint add voltage reference,"
- moved on the sheet: J22

Commit message: Signed-off-by: lokimetasmith <lokimail@gmail.com>
Parts:
- added R27, R29, R31, R36, R38, R39: 1000, Resistor_SMD:R_0805_2012Metric, symbol Device:R
- added R28, R35, R37, R40: 3K9, Resistor_SMD:R_0805_2012Metric, symbol Device:R
- added U10, U11: OP07, symbol Amplifier_Operational:OP07
- added U9: MCP4822, Package_SO:SOIC-8-1EP_3.9x4.9mm_P1.27mm_EP2.29x3mm, symbol Analog_DAC:MCP4822
Connections:
- net GND: now also R27.2, U10.3 (+), U11.3 (+), U9.7 (Vss)
- net GNDA: now also U6.3 (IN-)
- net VDDA: now also U3.4 (V-)
- net VSSA: no longer U3.4 (V-)
- net Vbias: now also R40.2, U11.6
- new net: R27.1, R28.1, R29.1
- new net: R31.1, U9.8 (VA)
- new net: R29.2, R31.2, R35.1, U10.2 (-)
- new net: R38.2, R39.2, R40.1, U11.2 (-)
- new net: R36.1, R37.1, R38.1
- new net +3V3: U9.1 (Vdd)
- new net +5V: U10.7 (V+), U11.7 (V+)
- new net -5V: R28.2, R37.2, U10.4 (V-), U11.4 (V-)
- new net >PORE: R35.2, U10.6
- new net CS_: U9.2 (~{CS})
- new net LDAC_: U9.5 (~{LDAC})
- new net SCK: U9.3 (SCK)
- new net SDI: U9.4 (SDI)
Other:
- note added: "-1.024V"
- note added: "-4V to 4V"
- note added: "0V to 2.048V"
- note added: "3K9 for plus and minus 4V 3.71093 for plus and minus 3.8V"
- note added: "I am leaning toward replacing this relatively primative OP07 with an OPA197. It's JFET input stage, low offset voltage, and rail-to-rail outputs are compelling selling points."
- note added: "Replace the 3K9 resistor with a 4K7 resistor in series with a 500 ohm trimpot for the full -5V ~ +5V range."
- note added: "The OP07 can swing to + and - 4V with this setup though + and - 3.8V is more reasonable. For this reason the notes describe amplification expansion of the 2.048V envelope of the DAC to 7.6V as well"
- note added: "Using an **Optically Isolated Current Source (LED + Photodiode)** is the "Ferrari" of dummy loads for nanopore amplifiers. While the resistor method (like in the EarlGrey PDF) is great for checking baseline noise, the LED/Photodiode method is superior for checking **bandwidth** and **step response** (simulating DNA events) because it solves the "Probe Capacitance" problem. Here is why the optical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"
- moved on the sheet: C10, C120, C121, C17, D82, J22, J7, NT2, R146, R8, TP11, U34

Commit message: Signed-off-by: lokimetasmith <lokimail@gmail.com>
Parts:
- removed R27, R29, R36, R38: 1000, Resistor_SMD:R_0805_2012Metric, symbol Device:R
- removed R28, R37: 3K9, Resistor_SMD:R_0805_2012Metric, symbol Device:R
- added U12, U13: ADR4550, Package_SO:SOIC-8_3.9x4.9mm_P1.27mm, symbol Reference_Voltage:ADR4550
Connections:
- net +5V: no longer U10.7 (V+)
- net -5V: no longer U10.4 (V-)
- net GND: no longer U10.3 (+), U9.7 (Vss)
- net GNDA: now also U10.2 (-), U9.7 (Vss), U12.4 (GND), U13.4 (GND)
- net VDDA: now also U10.7 (V+), U12.2 (IN), U13.2 (IN)
- net VSSA: now also U10.4 (V-)
- net at R31.2, R35.1: now also U10.3 (+), U13.6 (OUT); no longer U10.2 (-)
- net at R39.2, R40.1, U11.2 (-): now also U12.6 (OUT)
Other:
- note added: "For high-speed nanopore sensing, the answer is definitive: **Do NOT tie them together.** You should use **Separate Voltage References** (or at least strictly buffered separate paths) for your ADC and your Bias Driver. Here is the engineering reality of why sharing a "Reference Rail" will introduce a mysterious noise floor that you can't filter out. ### 1. The "Bully" on the Bus: The SAR ADC The 1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"
- note added: "consider cat 7 flat ribbon cable, 8 pairs, shielded"
- note added: "use a precision reference here"

Commit message: Signed-off-by: lokimetasmith <lokimail@gmail.com>
Parts:
- removed C46, C47: 0.1u, Capacitor_SMD:C_0603_1608Metric, symbol Device:C_Small
- removed JP2: Jumper_2_Bridged, symbol Jumper:Jumper_2_Bridged
- removed R10, R13: 27, Resistor_SMD:R_0402_1005Metric, symbol Device:R_Small_US
- added NT3: NetTie_2, NetTie:NetTie-2_SMD_Pad0.5mm, symbol Device:NetTie_2
- J5: footprint (none) -> Connector_JST:JST_PH_B5B-PH-K_1x05_P2.00mm_Vertical
- J6: footprint (none) -> Connector_JST:JST_PH_S5B-PH-K_1x05_P2.00mm_Horizontal
Connections:
- net USB_D+ is gone; now on net GPIO20: R15.2
- net USB_D- is gone; now on net GPIO19: R16.2
- net GUARD: now also NT3.1
- net Vbias: now also NT3.2
- net at C14.1, R18.1, U5.1 (IN)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: now also U1.6 (OUT-)

Commit message: Signed-off-by: lokimetasmith <lokimail@gmail.com>
Parts:
- added R10, R13, R27, R28: 1K, Resistor_SMD:R_0402_1005Metric, symbol Device:R
- added U14: TMUX1108RSV, Package_DFN_QFN:UQFN-16_1.8x2.6mm_P0.4mm, symbol Analog_Switch:TMUX1108RSV
- C1, C10, C118, C119, C120, C121, C13, C14, C15, C18, C2, C3, C4, C5, C6, C7: footprint Capacitor_SMD:C_0805_2012Metric -> Capacitor_SMD:C_0402_1005Metric
- C11, C12, C43, C44, C45, C75, C8, C9: footprint Capacitor_SMD:C_0603_1608Metric -> Capacitor_SMD:C_0402_1005Metric
- C16, C17: footprint Capacitor_SMD:C_1206_3216Metric -> Capacitor_SMD:C_0402_1005Metric
- R1: footprint Resistor_SMD:R_1206_3216Metric -> Resistor_SMD:R_0402_1005Metric
- R19, R2, R20, R21, R22, R3, R31, R35, R39, R4, R40, R5, R6, R7: footprint Resistor_SMD:R_0805_2012Metric -> Resistor_SMD:R_0402_1005Metric
Other:
- note added: "No, the schematic recipe I provided above is **Fixed Gain (10x)**. It uses a standard resistor, so the zoom level is locked. Since you are removing the MAX9939 (which *was* a variable gain amplifier), you likely want to keep that functionality—especially since Nanopores vary wildly in current. A 1 nA pore needs different gain than a 100 pA pore. Here is how to build a **"Safe" Variable Gain Ampli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"
