File: MR1/MR1.kicad_sch (KiCad schematic)
At the start: 106 parts, among them J1 Conn_Coaxial, J2 Conn_Coaxial, J22 B4B_PH, J23 Jumper_1, J3 USB_C_Receptacle_USB2.0, J36 Conn_ARM_JTAG_SWD_10, J4 Conn_Coaxial, J5 Conn_01x05_Socket, J6 Conn_01x05_Socket, J7 DIN-5_180degree, SW1 SW_Push, SW2 SW_Push, U1 LM27762, U10 OP07, U11 OP07, U12 ADR4550, U13 ADR4550, U14 TMUX1108RSV, U2 LMP7721, U3 OP07, U33 NCP163ASN330T1G, U34 NCP163ASN330T1G, U4 LT3045xDD, U5 LT3094xDD, U6 MCP3301, U7 SN65220, U8 ESP32-S3-MINI-1U, U9 MCP4822, Y2 32.768 kHz

Commit message: Signed-off-by: lokimetasmith <lokimail@gmail.com>
Parts:
- removed J2: Conn_Coaxial, Connector_Coaxial:MMCX_Molex_73415-0961_Horizontal_1.0mm-PCB, symbol Connector:Conn_Coaxial
- removed R8: 100K, Resistor_SMD:R_0402_1005Metric, symbol temp-sensor-rescue:R_Small_US-Device-temp-sensor-rescue
Connections:
- net SDI is gone; now on net CS_: U9.4 (SDI)
- net Signal: now also U14.6 (D)
- net at U14.2 (S1): now also R10.1
- net at U14.3 (S2): now also R13.1
- net at U14.4 (S3): now also R27.1
- net at U14.5 (S4): now also R28.1
- net at R13.2: now also R10.2, R27.2, R28.2
Other:
- moved on the sheet: C1, C10, C11, C118, C119, C12, C120, C121, C13, C14, C15, C16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

Commit message: Signed-off-by: lokimetasmith <lokimail@gmail.com>
Parts:
- removed J1, J4: Conn_Coaxial, Connector_Coaxial:MMCX_Molex_73415-0961_Horizontal_1.0mm-PCB, symbol Connector:Conn_Coaxial
- added J1, J2: Conn_01x01_Pin, footprints:Electrode, symbol Connector:Conn_01x01_Pin
- J6: footprint Connector_JST:JST_PH_S5B-PH-K_1x05_P2.00mm_Horizontal -> Connector_JST:JST_PH_S5B-PH-SM4-TB_1x05-1MP_P2.00mm_Horizontal
- U14: value TMUX1108RSV -> TMUX1104dgsr; footprint Package_DFN_QFN:UQFN-16_1.8x2.6mm_P0.4mm -> Package_SO:VSSOP-10_3x3mm_P0.5mm; symbol Analog_Switch:TMUX1108RSV -> MR1:TMUX1104DSG; LCSC (none) -> C2879206
- U2: LCSC (none) -> C124427
Connections:
- net ESP32_VCC_3V3: now also U14.5 (EN), U14.6 (VDD)
- net GNDA: now also U14.3 (GND)
- net GPIO40: now also U14.1 (A0)
- net GPIO41: now also U14.10 (A1)
- net Signal: now also C1.1, R1.1, U2.4; no longer J5.1 (Pin_1), R3.1, U14.6 (D), U3.6
- net at C1.2, R1.2, U2.8 (-): now also J1.1 (Pin_1)
- net at R6.2: now also J2.1 (Pin_1)
- net at R13.1: now also U14.9 (S2); no longer U14.3 (S2)
- net at R28.1: now also U14.7 (S4); no longer U14.5 (S4)
- net Signal_Return: now reaches U14.8 (D)
- net Signal_Return: now also J5.1 (Pin_1), R2.2
- new net: R3.1, U3.6
Other:
- moved on the sheet: C1, C6, J5, J6, R1, R2, R3, R4, R5, R6, U2, U3

Commit message: Signed-off-by: lokimetasmith <lokimail@gmail.com>
Parts:
- added J4: Conn_01x08, 4ms_Connector:Pins_1x08_2.54mm_TH, symbol PCM_4ms_Connector:Conn_01x08
Connections:
- net >PORE: now also J4.8 (Pin_8)
- net GNDA: now also J4.1 (Pin_1), J4.4 (Pin_4), J4.7 (Pin_7)
- net Signal: now also J4.2 (Pin_2)
- net VDDA: now also J4.3 (Pin_3)
- net VSSA: now also J4.6 (Pin_6)
- net Vbias: now also J4.5 (Pin_5)
- net at R3.1, U3.6: now also U6.2 (IN+)
Other:
- moved on the sheet: U6

Commit message: Signed-off-by: lokimetasmith <lokimail@gmail.com>
Parts:
- removed J4: Conn_01x08, 4ms_Connector:Pins_1x08_2.54mm_TH, symbol PCM_4ms_Connector:Conn_01x08
- removed J5: Conn_01x05_Socket, Connector_JST:JST_PH_B5B-PH-K_1x05_P2.00mm_Vertical, symbol Connector:Conn_01x05_Socket
- removed J6: Conn_01x05_Socket, Connector_JST:JST_PH_S5B-PH-SM4-TB_1x05-1MP_P2.00mm_Horizontal, symbol Connector:Conn_01x05_Socket
- removed R2: 100, Resistor_SMD:R_0402_1005Metric, symbol Device:R
- added J10, J11: Conn_01x01_Pin, footprints:Electrode, symbol Connector:Conn_01x01_Pin
- added J12, J9: Conn_01x10, Connector_JST:JST_SH_SM10B-SRSS-TB_1x10-1MP_P1.00mm_Horizontal, symbol MR1:Conn_01x11_MP
- added NT4: NetTie_2, NetTie:NetTie-2_SMD_Pad0.5mm, symbol Device:NetTie_2
- added R8: 100, Resistor_SMD:R_0402_1005Metric, symbol Device:R
Connections:
- net >PORE: now also J12.7 (Pin_7)
- net GNDA: now also J12.3 (Pin_3), J12.6 (Pin_6), J12.8 (Pin_8), J9.10 (Pin_10), J9.3 (Pin_3), J9.5 (Pin_5), J9.7 (Pin_7)
- net Signal_Return: now also R5.1, U3.3 (+), J12.2 (Pin_2)
- net VDDA: now also J12.5 (Pin_5), J9.9 (Pin_9)
- net VSSA: now also J12.4 (Pin_4), J9.8 (Pin_8)
- net Vbias: now also J12.9 (Pin_9), NT4.1; no longer C6.1, NT3.2, R6.1, U2.1 (+)
- net Signal: no longer names the net of C1.1, R1.1, U2.4
- net Signal: now also R8.2
- new net >PORE_AMP: J10.1 (Pin_1), J9.2 (Pin_2)
- new net SHIELD: J12.1 (Pin_1), J12.10 (Pin_10), J12.MP (Pin_11), NT4.2
- new net SHIELD_AMP: J9.1 (Pin_1), J9.MP (Pin_11)
- new net Signal_AMP: J9.6 (Pin_6), R8.1
- new net Vbias_AMP: C6.1, J11.1 (Pin_1), J9.4 (Pin_4), NT3.2, R6.1, U2.1 (+)
Other:
- note added: "250ft 32AWG CAT7 STP Solid, 0.075" Super Flat Bulk Ethernet Bare Copper Cable - White."
- note added: "P1"
- note added: "P2"
- note added: "P3"
- note added: "P4"
- note added: "SHR-10V-S"
- note added: "SM10B-SRSS-TB"
- note added: "SSH-003T-P0.2-H #32 to #28 (0.032 to 0.081) 0.4 to 0.8 23,000"
- note added: "amplifier board"
- note added: "https://www.vpi.us/bulk-cable-sf/super-flat-cat7-736#idTab9"
- moved on the sheet: C2, C3, C4, C5, NT3, R3, R31, R35, R39, R4, R40, R5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

Commit message: added nanopore depression, updated cad
Signed-off-by: lokimetasmith <lokimail@gmail.com>
Parts:
- added H1: Nanopore, footprints:Nanopore holder_recessed, symbol Mechanical:MountingHole
Connections:
- net >PORE: now also J12.2 (Pin_2); no longer J12.7 (Pin_7)
- net GNDA: now also J12.5 (Pin_5), J12.7 (Pin_7); no longer J12.6 (Pin_6), J12.8 (Pin_8)
- net GPIO38: no longer R130.1
- net GPIO40: now also R43.1; no longer U14.1 (A0)
- net GPIO41: now also R130.1; no longer U14.10 (A1)
- net GPIO7: no longer R43.1
- net Signal_Return: now also J12.6 (Pin_6), R3.1, U3.6, U6.2 (IN+); no longer J12.2 (Pin_2)
- net VDDA: now also J12.9 (Pin_9); no longer J12.5 (Pin_5)
- net VSSA: now also J12.8 (Pin_8); no longer J12.4 (Pin_4)
- net Vbias: now also J12.4 (Pin_4), R10.2, R13.2, R27.2, R28.2; no longer J12.9 (Pin_9)
- net at U9.6 (VB): now also R39.1
- net TMUX_A0: now reaches R43.2
- net TMUX_A0: now also U14.1 (A0)
- net TMUX_A1: now reaches R130.2
- net TMUX_A1: now also U14.10 (A1)
- net DIN renamed GPIO18
- net Fan_0_PWM renamed GPIO12
- net Fan_0_Tach renamed GPIO5
- net Fan_1_PWM renamed GPIO13
- net Fan_2_PWM renamed GPIO14
- net Fan_EN renamed GPIO11
Other:
- note added: "pins for holding the board in place while applying adhesive https://www.mcmaster.com/98378A208/"
- moved on the sheet: C10, C120, C121, C17, C51, C52, D82, J3, R10, R11, R12, R13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

Commit message: Signed-off-by: lokimetasmith <lokimail@gmail.com>
Parts:
- removed C43, C44, C45, C75, C8: 0.1u, Capacitor_SMD:C_0402_1005Metric, symbol Device:C_Small
- removed R19, R20, R21, R22: 5k, Resistor_SMD:R_0402_1005Metric, symbol Device:R
- removed R31, R39: 1000, Resistor_SMD:R_0402_1005Metric, symbol Device:R
- removed U3: OP07, Package_SO:SOIC-8_3.9x4.9mm_P1.27mm, symbol Amplifier_Operational:OP07
- added C19, C20: 100nF, Capacitor_SMD:C_0402_1005Metric, symbol Device:C
- added C21, C22: 22u, Capacitor_SMD:C_0402_1005Metric, symbol Device:C_Small
- added C23, C8: 4.7u, Capacitor_SMD:C_0402_1005Metric, symbol temp-sensor-rescue:C_Small-Device-temp-sensor-rescue
- added R19: 9.16k, Resistor_SMD:R_0402_1005Metric, symbol Device:R_Small_US
- added R2: 24.9k 0.1%, Resistor_SMD:R_0402_1005Metric, symbol Device:R
- added R20: 9.09k, Resistor_SMD:R_0402_1005Metric, symbol Device:R_Small_US
- added R21, R22, R29, R36: 10k 1%, Resistor_SMD:R_0402_1005Metric, symbol Device:R_Small_US
- added U16: LTC6268xS8-10, Package_SO:SO-8_3.9x4.9mm_P1.27mm, symbol MR1:LTC6268xS8-10_SHIELD
- R7: value 5k -> 24.9k 0.1%
- U4: footprint Package_DFN_QFN:DFN-10-1EP_3x3mm_P0.5mm_EP1.65x2.38mm -> Package_DFN_QFN:DFN-12-1EP_3x3mm_P0.5mm_EP1.6x2.5mm; symbol Regulator_Linear:LT3045xDD -> MR1:LT3045xDD-1
Connections:
- net +5V is gone; now on net VDDA: U11.7 (V+)
- net -5V is gone; now on net VSSA: U11.4 (V-)
- net GNDA: now also J12.10 (Pin_10), R7.2, U4.6 (ILIM), U4.9 (GND), U5.6 (ILIM), C19.2, C20.2, C21.1, C22.1, C23.1, C8.1, R2.2; no longer U4.8 (GND)
- net SHIELD: no longer J12.10 (Pin_10)
- net Signal_Return: now also U16.3 (+); no longer R3.1, U6.2 (IN+)
- net VDDA: now also U4.11 (OUT), U4.12 (OUT), C19.1, C21.2, U16.7 (V+); no longer U4.9 (OUTS)
- net VSSA: now also U5.11 (OUT), U5.12 (OUT), C20.1, C22.2, U16.5 (V-)
- net Vbias: now also U6.1 (Vref), U16.1 (NC), U16.4 (NC)
- net at R3.2, R4.2: now also U16.2 (-)
- net +Vp: now reaches C15.2, R24.2, U1.11 (OUT+), U4.1 (IN), U4.2 (IN)
- net +Vp: now also U4.4 (EN/UV), U4.7 (PGFB)
- net at U9.8 (VA): now also R36.2
- net at R35.1, U10.3 (+): now also R29.1, R36.1; no longer U13.6 (OUT)
- net -Vp: now reaches C14.1, R18.1, U1.6 (OUT-), U5.1 (IN), U5.13 (IN), U5.2 (IN)
- net -Vp: now also U5.3 (EN/UV), U5.5 (PGFB)
- net FB-: now reaches R18.2, R26.1, U1.7 (FB-)
- net FB-: now also R20.2
- net at R40.1, U11.2 (-): now also R21.1, R22.1; no longer U12.6 (OUT)
- net +VIOC: now reaches U4.3 (VIOC)
- net +VIOC: now also R19.1
- net FB+: now reaches R24.1, R25.2, U1.2 (FB+)
- net FB+: now also R19.2
- net at R7.1: now also U5.8 (SET), C23.2
- net at U9.6 (VB): now also R21.2
- net -VIOC: now reaches U5.7 (VIOC)
- net -VIOC: now also R20.1
- net at U1.12 (EN+): now also U1.8 (EN-)
- new net: R3.1, U16.6, U6.2 (IN+)
- new net: R29.2, U13.6 (OUT)
- new net: C8.2, R2.1, U4.8 (SET)
- new net: R22.2, U12.6 (OUT)
Other:
- note added: "3045-1"
- note added: "LTC6268, alternate to TI's opamp"
- note added: "PGA855"
- note added: "Stability in ultra-low noise regulators is dictated by the **Output Capacitance ()** and the **Noise Reduction Capacitance ()**. If these ratios are wrong, the LDO will oscillate, turning your "clean" power supply into a radio transmitter. ### 1. The LDO Component Values (The Critical Stage) These regulators do not use standard voltage dividers. They use a precision current source architecture. Y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"
- note added: "Stage 1: Transimpedance Amp"
- note added: "Virtual Ground"
- note added: "place R19 and R20 or place R18 and R24, not both."
- note removed: "ADC1 is recommended for use."
- note removed: "OPA189"
- note removed: "Stability in ultra-low noise regulators is dictated by the **Output Capacitance ()** and the **Noise Reduction Capacitance ()**. If these ratios are wrong, the LDO will oscillate, turning your "clean" power supply into a radio transmitter. Here are the exact calculated values and part types you need for the **TPS7A94 (Positive)** and **LT3094 (Negative)**, assuming a +/- 6.5V raw supply to get a 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"
- note removed: "When ATTEN=2 and the effective measurement range is 0 ~ 1600 mV, the total error is ±10 mV."
- moved on the sheet: NT4, R10, R13, R18, R23, R24, R25, R26, R27, R28, U14

Commit message: Signed-off-by: lokimetasmith <lokimail@gmail.com>
Parts:
- removed R36: 10k 1%, Resistor_SMD:R_0402_1005Metric, symbol Device:R_Small_US
- added R31: 3K9, Resistor_SMD:R_0402_1005Metric, symbol Device:R
Connections:
- net >PORE: now also J12.1 (Pin_1), R29.1; no longer J12.2 (Pin_2), R35.2
- net >PORE_AMP: now also J9.1 (Pin_1); no longer J9.2 (Pin_2)
- net GNDA: now also J12.2 (Pin_2), J12.6 (Pin_6), J9.2 (Pin_2), J9.6 (Pin_6); no longer J12.10 (Pin_10), J12.3 (Pin_3), J12.5 (Pin_5), J12.7 (Pin_7), J9.10 (Pin_10), J9.3 (Pin_3), J9.5 (Pin_5), J9.7 (Pin_7)
- net SHIELD: now also J12.10 (Pin_10), J12.4 (Pin_4), J12.9 (Pin_9); no longer J12.1 (Pin_1)
- net SHIELD_AMP: now also J9.10 (Pin_10), J9.4 (Pin_4), J9.9 (Pin_9); no longer J9.1 (Pin_1)
- net Signal_AMP: now also J9.5 (Pin_5); no longer J9.6 (Pin_6)
- net Signal_Return: now also J12.5 (Pin_5); no longer J12.6 (Pin_6)
- net VDDA: now also J12.8 (Pin_8), J9.7 (Pin_7); no longer J12.9 (Pin_9), J9.9 (Pin_9)
- net VSSA: now also J12.7 (Pin_7); no longer J12.8 (Pin_8)
- net Vbias: now also J12.3 (Pin_3); no longer J12.4 (Pin_4)
- net Vbias_AMP: now also J9.3 (Pin_3); no longer J9.4 (Pin_4)
- net at C7.1, NT1.2, R9.1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: now also C119.1
- net at R29.2: now also R35.2, U10.3 (+), R31.2; no longer U13.6 (OUT)
- net at U9.8 (VA): now also R31.1
- net at NT1.1, U33.5 (VOUT): no longer C119.1
- new net: R35.1, U13.6 (OUT)
Other:
- note added: "-2.4V to 2.4V"
- moved on the sheet: C119, J1, J12, J2, J9, R29

Commit message: Signed-off-by: lokimetasmith <lokimail@gmail.com>
Parts:
- removed C1: 2pF, Capacitor_SMD:C_0402_1005Metric, symbol Device:C
- removed C10, C13, C14, C15, C18, C23, C8: 4.7u, Capacitor_SMD:C_0402_1005Metric, symbol temp-sensor-rescue:C_Small-Device-temp-sensor-rescue
- removed C11, C12: 0.1u, Capacitor_SMD:C_0402_1005Metric, symbol Device:C_Small
- removed C118, C119, C120, C121, C7: 10u, Capacitor_SMD:C_0402_1005Metric, symbol Device:C_Small
- removed C16, C17: 10u, Capacitor_SMD:C_0402_1005Metric, symbol temp-sensor-rescue:C_Small-Device-temp-sensor-rescue
- removed C19, C2, C20, C3, C6: 100nF, Capacitor_SMD:C_0402_1005Metric, symbol Device:C
- removed C21, C22: 22u, Capacitor_SMD:C_0402_1005Metric, symbol Device:C_Small
- removed C4, C5: 10nF, Capacitor_SMD:C_0402_1005Metric, symbol Device:C
- removed C51, C52: 12p, Capacitor_SMD:C_0402_1005Metric, symbol Device:C_Small
- removed C9: 4.7u, Capacitor_SMD:C_0402_1005Metric, symbol Device:C_Small
- removed D82: MBR0540, Diode_SMD:D_SOD-123, symbol Diode:MBR0540
- removed H1: Nanopore, footprints:Nanopore holder_recessed, symbol Mechanical:MountingHole
- removed J1, J10, J11, J2: Conn_01x01_Pin, footprints:Electrode, symbol Connector:Conn_01x01_Pin
- removed J12, J9: Conn_01x10, Connector_JST:JST_SH_SM10B-SRSS-TB_1x10-1MP_P1.00mm_Horizontal, symbol MR1:Conn_01x11_MP
- removed J22: B4B_PH, Connector_JST:JST_PH_B4B-PH-K_1x04_P2.00mm_Vertical, symbol Connector_Generic:Conn_01x04
- removed J23: Jumper_1, Connector_PinHeader_2.54mm:PinHeader_1x02_P2.54mm_Vertical, symbol Connector:Conn_01x02_Pin
- removed J3: USB_C_Receptacle_USB2.0, Connector_USB:USB_C_Receptacle_HRO_TYPE-C-31-M-12, symbol Connector:USB_C_Receptacle_USB2.0
- removed J36: Conn_ARM_JTAG_SWD_10, Connector_PinHeader_1.27mm:PinHeader_2x05_P1.27mm_Vertical_SMD, symbol Connector:Conn_ARM_JTAG_SWD_10
- removed J7: DIN-5_180degree, symbol Connector:DIN-5_180degree
- removed NT1, NT2, NT3, NT4: NetTie_2, NetTie:NetTie-2_SMD_Pad0.5mm, symbol Device:NetTie_2
- removed R1: 1M, Resistor_SMD:R_0402_1005Metric, symbol Device:R
- removed R10, R13, R27, R28, R3, R5, R6: 1K, Resistor_SMD:R_0402_1005Metric, symbol Device:R
- removed R11, R12: 15K, Resistor_SMD:R_0402_1005Metric, symbol temp-sensor-rescue:R_Small_US-Device-temp-sensor-rescue
- removed R130, R143, R43, R96, R97: 27, Resistor_SMD:R_0402_1005Metric, symbol Device:R_Small_US
- removed R14, R17: 5.1k, Resistor_SMD:R_0402_1005Metric, symbol temp-sensor-rescue:R_Small_US-Device-temp-sensor-rescue
- removed R145, R146: 10k, Resistor_SMD:R_0402_1005Metric, symbol Device:R
- removed R15, R16: 27, Resistor_SMD:R_0402_1005Metric, symbol temp-sensor-rescue:R_Small_US-Device-temp-sensor-rescue
- removed R18, R21, R22, R23, R24, R25, R26, R29, R33, R34, R9: 10k 1%, Resistor_SMD:R_0402_1005Metric, symbol Device:R_Small_US
- removed R19: 9.16k, Resistor_SMD:R_0402_1005Metric, symbol Device:R_Small_US
- removed R2, R7: 24.9k 0.1%, Resistor_SMD:R_0402_1005Metric, symbol Device:R
- removed R20: 9.09k, Resistor_SMD:R_0402_1005Metric, symbol Device:R_Small_US
- removed R30: 1M, Resistor_SMD:R_0402_1005Metric, symbol Device:R_Small_US
- removed R31, R35, R40: 3K9, Resistor_SMD:R_0402_1005Metric, symbol Device:R
- removed R32, R51: 0, Resistor_SMD:R_0402_1005Metric, symbol Device:R_Small_US
- removed R4, R8: 100, Resistor_SMD:R_0402_1005Metric, symbol Device:R
- removed SW1, SW2: SW_Push, Custom Footprints:SW_SPST_6mm_gull wing, symbol Switch:SW_Push
- removed TP11: TestPoint, TestPoint:TestPoint_Pad_D1.0mm, symbol Connector:TestPoint
- removed U1: LM27762, Package_SON:WSON-12-1EP_3x2mm_P0.5mm_EP1x2.65_ThermalVias, symbol Regulator_SwitchedCapacitor:LM27762
- removed U10, U11: OP07, symbol Amplifier_Operational:OP07
- removed U12, U13: ADR4550, Package_SO:SOIC-8_3.9x4.9mm_P1.27mm, symbol Reference_Voltage:ADR4550
- removed U14: TMUX1104dgsr, Package_SO:VSSOP-10_3x3mm_P0.5mm, symbol MR1:TMUX1104DSG
- removed U16: LTC6268xS8-10, Package_SO:SO-8_3.9x4.9mm_P1.27mm, symbol MR1:LTC6268xS8-10_SHIELD
- removed U2: LMP7721, Package_SO:SOIC-8_3.9x4.9mm_P1.27mm, symbol LMP7721:LMP7721
- removed U33, U34: NCP163ASN330T1G, Package_TO_SOT_SMD:SOT-23-5, symbol Regulator_Linear:NCP163ASN330T1G
- removed U4: LT3045xDD, Package_DFN_QFN:DFN-12-1EP_3x3mm_P0.5mm_EP1.6x2.5mm, symbol MR1:LT3045xDD-1
- removed U5: LT3094xDD, Package_DFN_QFN:DFN-12-1EP_3x3mm_P0.45mm_EP1.65x2.38mm_ThermalVias, symbol Regulator_Linear:LT3094xDD
- removed U6: MCP3301, symbol Analog_ADC:MCP3301
- removed U7: SN65220, Package_TO_SOT_SMD:SOT-23-6, symbol twig:SN65220-Power_Protection_passthrough
- removed U8: ESP32-S3-MINI-1U, RF_Module:ESP32-S2-MINI-1U, symbol RF_Module:ESP32-S3-MINI-1U
- removed U9: MCP4822, Package_SO:SOIC-8-1EP_3.9x4.9mm_P1.27mm_EP2.29x3mm, symbol Analog_DAC:MCP4822
- removed Y2: 32.768 kHz, Crystal:Crystal_SMD_3215-2Pin_3.2x1.5mm, symbol Device:Crystal
- added C28: 2pF, Capacitor_SMD:C_0402_1005Metric, symbol Device:C
- added E1: SparkGap, symbol Device:SparkGap
- added H2, H3, H4, H5, H6, H7, H8, H9: MountingHole_Pad, symbol Mechanical:MountingHole_Pad
- added R38: 1M, Resistor_SMD:R_0402_1005Metric, symbol Device:R
Connections:
- net GNDA: now also C28.1, E1.2, H2.1, H3.1, H4.1, H5.1, R38.1
- new net Earth: C28.2, E1.1, H6.1, H7.1, H8.1, H9.1, R38.2
- no-connect marks 2 -> 0
Other:
- sheet Ignition ports: added >PORE; removed none
- sheet Insturmentation ports: added >PORE, Vbias; removed none
- sheet Microcontroller ports: added RXD0, TXD0, USB_D+, USB_D-; removed none
- sheet Power ports: added USB_D+, USB_D-; removed none
- note removed: "+VOUT = 1.2 V × (R1 + R2) / R2 -VOUT = -1.22 V × (R3 + R4) / R4"
- note removed: "-1.024V"
- note removed: "-2.4V to 2.4V"
- note removed: "-4V to 4V"
- note removed: "0V to 2.048V"
- note removed: "250ft 32AWG CAT7 STP Solid, 0.075" Super Flat Bulk Ethernet Bare Copper Cable - White."
- note removed: "3. Selecting the Precision ADC To capture <1µV signals, you need a 24-bit or 32-bit Delta-Sigma ADC. The standard 12-bit or 16-bit SAR ADCs used in microcontrollers will not see the signal floor you have created. Top Recommendations: TI ADS1261 (24-bit / 32-bit mode): Why: It has a built-in PGA (Programmable Gain Amplifier) that is extremely low noise. Noise Floor: Can resolve down to ~6 nV RMS a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"
- note removed: "3045-1"
- note removed: "3K9 for plus and minus 4V 3.71093 for plus and minus 3.8V"
- note removed: "499Ω Metal Film Resistor"
- note removed: "9.0PF"
- note removed: "ADC1: 10 channels: GPIO1 - GPIO10 ADC2 is shared with WiFi"
- note removed: "Boot Mode | GPIO0 | GPIO46 Default Config | 1(pull-up)| 0 (Pull-down) SPI Boot | 1 | Any Value Joint DL Boot | 0 | 0 Invalid | 0 | 1"
- note removed: "C2 and C3 X5R"
- note removed: "ESD"
- note removed: "I am leaning toward replacing this relatively primative OP07 with an OPA197. It's JFET input stage, low offset voltage, and rail-to-rail outputs are compelling selling points."
- note removed: "Jumper"
- note removed: "LTC6268"
- note removed: "LTC6268, alternate to TI's opamp"
- note removed: "MCP33131"
- note removed: "MG Chemicals 422C conformal coating"
- note removed: "No, the schematic recipe I provided above is **Fixed Gain (10x)**. It uses a standard resistor, so the zoom level is locked. Since you are removing the MAX9939 (which *was* a variable gain amplifier), you likely want to keep that functionality—especially since Nanopores vary wildly in current. A 1 nA pore needs different gain than a 100 pA pore. Here is how to build a **"Safe" Variable Gain Ampli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"
- note removed: "P1"
- note removed: "P2"
- note removed: "P3"
- note removed: "P4"
- note removed: "PGA855"
- note removed: "PTFE (ZYF255DA): Dk .approx 2.55"
- note removed: "R1 1206"
- note removed: "Replace the 3K9 resistor with a 4K7 resistor in series with a 500 ohm trimpot for the full -5V ~ +5V range."
- note removed: "SHR-10V-S"
- note removed: "SM10B-SRSS-TB"
- note removed: "SSH-003T-P0.2-H #32 to #28 (0.032 to 0.081) 0.4 to 0.8 23,000"
- note removed: "Stage 1: Transimpedance Amp"
- note removed: "TPS7A94"
- note removed: "The OP07 can swing to + and - 4V with this setup though + and - 3.8V is more reasonable. For this reason the notes describe amplification expansion of the 2.048V envelope of the DAC to 7.6V as well"
- note removed: "UART TTL or SPI, selectable in firmware"
- note removed: "Virtual Ground"
- note removed: "Y2: ESR = Max. 70 KΩ 32.768 kHz"
- note removed: "amplifier board"
- note removed: "consider cat 7 flat ribbon cable, 8 pairs, shielded"
- note removed: "https://www.vpi.us/bulk-cable-sf/super-flat-cat7-736#idTab9"
- note removed: "low noise voltage converters"
- note removed: "pins for holding the board in place while applying adhesive https://www.mcmaster.com/98378A208/"
- note removed: "place R19 and R20 or place R18 and R24, not both."
- note removed: "use a precision reference here"
