File: MR1/MR1.kicad_sch (KiCad schematic)
At the start: 11 parts

Commit message: Signed-off-by: lokimetasmith <lokimail@gmail.com>
Parts:
- H2, H3, H4, H5: footprint (none) -> MountingHole:MountingHole_6mm_Pad_Via
- H6, H7, H8, H9: footprint (none) -> MountingHole:MountingHole_3.2mm_M3_Pad_Via
Other:
- sheet Ignition ports: added CS_, LDAC_, SCK, SDI; removed none
- sheet Insturmentation ports: added DAC_CLK, DAC_Dout, DAC_EN; removed Vbias
- sheet Microcontroller ports: added CS_, DAC_CLK, DAC_Dout, DAC_EN, LDAC_, SCK, SDI; removed none

Commit message: Signed-off-by: lokimetasmith <lokimail@gmail.com>
Parts:
- added C36: 2pF, Capacitor_SMD:C_0402_1005Metric, symbol Device:C
- added E2: SparkGap, symbol Device:SparkGap
- added R47: 1M, Resistor_SMD:R_0402_1005Metric, symbol Device:R
Connections:
- net Earth: now also C36.2, E2.1, R47.2
- new net GND: C36.1, E2.2, R47.1
Other:
- note added: "TODO List : Done: update ADC with correct library part and footprint add voltage reference, Look at Insturmentation amplifiers Remaining: flip board around, route tubing on the underside of the board. punch through the back side with a via to the sensitized silver chloride pad, which reduces a potential liquid contact point over solder mask/conformal."
- note removed: "Add precision low noise ADC"
- note removed: "Look at Insturmentation amplifiers"
- note removed: "TODO: update ADC with correct library part and footprint add voltage reference,"
