File: MR1/MR1.kicad_pcb (KiCad board)
At the start: 6 copper layers, 8.8 x 8.8 mm, 104 parts, among them J1 Conn_01x01_Pin, J10 Conn_01x01_Pin, J11 Conn_01x01_Pin, J12 Conn_01x10, J2 Conn_01x01_Pin, J22 B4B_PH, J23 Jumper_1, J3 USB_C_Receptacle_USB2.0, J36 Conn_ARM_JTAG_SWD_10, J9 Conn_01x10, U1 LM27762, U12 ADR4550, U13 ADR4550, U14 TMUX1104dgsr, U16 LTC6268xS8-10, U2 LMP7721, U33 NCP163ASN330T1G, U34 NCP163ASN330T1G, U4 LT3045xDD, U5 LT3094xDD, U7 SN65220, U8 ESP32-S3-MINI-1U, U9 MCP4822, Y2 32.768 kHz

Commit message: Signed-off-by: lokimetasmith <lokimail@gmail.com>
Parts:
- removed C1: 2pF, Capacitor_SMD:C_0402_1005Metric
- removed C120: 10u, Capacitor_SMD:C_0402_1005Metric
- removed C2, C3, C6: 100nF, Capacitor_SMD:C_0402_1005Metric
- removed C4, C5: 10nF, Capacitor_SMD:C_0402_1005Metric
- removed H1: Nanopore, footprints:Nanopore holder_recessed
- removed J1, J10, J11, J2: Conn_01x01_Pin, footprints:Electrode
- removed J9: Conn_01x10, Connector_JST:JST_SH_SM10B-SRSS-TB_1x10-1MP_P1.00mm_Horizontal
- removed NT3: NetTie_2, NetTie:NetTie-2_SMD_Pad0.5mm
- removed R1: 1M, Resistor_SMD:R_0402_1005Metric
- removed R10, R13, R27, R28, R6: 1K, Resistor_SMD:R_0402_1005Metric
- removed R146: 10k, Resistor_SMD:R_0402_1005Metric
- removed R22, R33: 10k 1%, Resistor_SMD:R_0402_1005Metric
- removed R40: 3K9, Resistor_SMD:R_0402_1005Metric
- removed R8: 100, Resistor_SMD:R_0402_1005Metric
- removed U12: ADR4550, Package_SO:SOIC-8_3.9x4.9mm_P1.27mm
- removed U14: TMUX1104dgsr, Package_SO:VSSOP-10_3x3mm_P0.5mm
- removed U2: LMP7721, Package_SO:SOIC-8_3.9x4.9mm_P1.27mm
- removed U34: NCP163ASN330T1G, Package_TO_SOT_SMD:SOT-23-5
- added C25: 100nF, Capacitor_SMD:C_0402_1005Metric, F.Cu at (98.1, 151.9)
- added C27: 100nF, Capacitor_SMD:C_0402_1005Metric, F.Cu at (98.1, 153.9)
- added C28: 2pF, Capacitor_SMD:C_0402_1005Metric, F.Cu at (42.7, 160.2)
- added R38: 1M, Resistor_SMD:R_0402_1005Metric, F.Cu at (42.7, 158.2)
- added U3: OPA197xD, Package_SO:SOIC-8_3.9x4.9mm_P1.27mm, F.Cu at (98.5, 116.7)
- C11, C12: value 0.1u -> 10nF
- R21: value 10k 1% -> 82k 1%
- moved J36 91.6 mm to (54.9, 121.9)
- moved C11 89.3 mm to (66.2, 132.3), turned to 180 degrees
- moved C12 82.9 mm to (66.2, 128.4), turned to 180 degrees
- moved C121 82.9 mm to (31.6, 134.0), turned to -90 degrees
- moved R21 74.0 mm to (97.8, 110.4), turned to 90 degrees
- moved U9 54.0 mm to (98.5, 104.8), turned to -90 degrees
- moved U13 52.8 mm to (105.2, 104.8), turned to -90 degrees
- moved R31 51.4 mm to (100.3, 110.4), turned to -90 degrees
- moved R35 12.9 mm to (102.4, 110.4)
- moved C9 5.88 mm to (66.1, 135.9)
- moved C119 4.51 mm to (37.5, 134.3)
Connections:
- net /+VIOC renamed /Power/+VIOC
- net /+Vp renamed /Power/+Vp
- net /-VIOC renamed /Power/-VIOC
- net /-Vp renamed /Power/-Vp
- net />PORE renamed /Ignition/>PORE
- net /CC1 renamed /Power/CC1
- net /CC2 renamed /Power/CC2
- net /D+ renamed /Power/D+
- net /D- renamed /Power/D-
- net /FB+ renamed /Power/FB+
- net /FB- renamed /Power/FB-
- net /GPIO1 renamed /Microcontroller/GPIO1
- net /GPIO10 renamed /Microcontroller/GPIO10
- net /GPIO11 renamed /Microcontroller/GPIO11
- net /GPIO12 renamed /Microcontroller/GPIO12
- net /GPIO13 renamed /Microcontroller/GPIO13
- net /GPIO14 renamed /Microcontroller/GPIO14
- net /GPIO15 renamed /Microcontroller/GPIO15
- net /GPIO16 renamed /Microcontroller/GPIO16
- net /GPIO17 renamed /Microcontroller/GPIO17
- net /GPIO18 renamed /Microcontroller/GPIO18
- net /GPIO19 renamed /Microcontroller/GPIO19
- net /GPIO2 renamed /Microcontroller/GPIO2
- net /GPIO20 renamed /Microcontroller/GPIO20
- net /GPIO21 renamed /Microcontroller/GPIO21
- net /GPIO26 renamed /Microcontroller/GPIO26
- net /GPIO3 renamed /Microcontroller/GPIO3
- net /GPIO33 renamed /Microcontroller/GPIO33
- net /GPIO34 renamed /Microcontroller/GPIO34
- net /GPIO35 renamed /Microcontroller/GPIO35
- net /GPIO36 renamed /Microcontroller/GPIO36
- net /GPIO37 renamed /Microcontroller/GPIO37
- net /GPIO38 renamed /Microcontroller/GPIO38
- net /GPIO39 renamed /Microcontroller/GPIO39
- net /GPIO4 renamed /Microcontroller/GPIO4
- net /GPIO40 renamed /Microcontroller/GPIO40
- net /GPIO41 renamed /Microcontroller/GPIO41
- net /GPIO42 renamed /Microcontroller/GPIO42
- net /GPIO45 renamed /Microcontroller/GPIO45
- net /GPIO46 renamed /Microcontroller/GPIO46
- net /GPIO47 renamed /Microcontroller/GPIO47
- net /GPIO48 renamed /Microcontroller/GPIO48
- net /GPIO5 renamed /Microcontroller/GPIO5
- net /GPIO6 renamed /Microcontroller/GPIO6
- net /GPIO7 renamed /Microcontroller/GPIO7
- net /GPIO8 renamed /Microcontroller/GPIO8
- net /GPIO9 renamed /Microcontroller/GPIO9
- net /JTAG_TCK renamed /Microcontroller/JTAG_TCK
- net /JTAG_TDI renamed /Microcontroller/JTAG_TDI
- net /JTAG_TDO renamed /Microcontroller/JTAG_TDO
- net /JTAG_TMS renamed /Microcontroller/JTAG_TMS
- net /RX renamed /Microcontroller/RX
- net /RXD0 renamed /Microcontroller/RXD0
- net /SHIELD renamed /Insturmentation/SHIELD
- net /Signal_Return renamed /Insturmentation/Signal_Return
- net /TX renamed /Microcontroller/TX
- net /TXD0 renamed /Microcontroller/TXD0
- net /V_USB renamed /Power/V_USB
- net /Vbias renamed /Insturmentation/Vbias
- net LDAC_ renamed /Ignition/LDAC_
- net SCK renamed /Ignition/SCK
- C11 pad 1: GND -> VDDA
- C11 pad 2: /CHIP_PU -> GNDA
- C119 pad 1: Net-(U8-3V3) -> /Microcontroller/VCC_3V3
- C12 pad 1: GND -> VSSA
- C12 pad 2: /GPIO0 -> GNDA
- C121 pad 1: ESP32_VCC_3V3 -> +3V3
- C7 pad 1: Net-(U8-3V3) -> /Microcontroller/VCC_3V3
- C9 pad 1: /CHIP_PU -> /Microcontroller/CHIP_PU
- J22 pad 1: ESP32_VCC_3V3 -> /Microcontroller/VCC_3V3
- J3 pad S1: GND -> Earth
- J36 pad 1: ESP32_VCC_3V3 -> /Microcontroller/VCC_3V3
- J36 pad 10: /CHIP_PU -> /Microcontroller/CHIP_PU
- NT1 pad 1: Net-(U33-VOUT) -> +3.3V
- NT1 pad 2: Net-(U8-3V3) -> /Microcontroller/VCC_3V3
- R130 pad 2: /TMUX_A1 -> /Microcontroller/TMUX_A1
- R143 pad 2: /GPIO0 -> /Microcontroller/GPIO0
- R21 pad 1: Net-(U11--) -> Net-(U3-+)
- R29 pad 2: Net-(U10-+) -> Net-(U3-+)
- R31 pad 2: Net-(U10-+) -> Net-(U3-+)
- R34 pad 1: ESP32_VCC_3V3 -> /Microcontroller/VCC_3V3
- R35 pad 2: Net-(U10-+) -> Net-(U3-+)
- R43 pad 2: /TMUX_A0 -> /Microcontroller/TMUX_A0
- R9 pad 1: Net-(U8-3V3) -> /Microcontroller/VCC_3V3
- R9 pad 2: /CHIP_PU -> /Microcontroller/CHIP_PU
- TP11 pad 1: ESP32_VCC_3V3 -> /Microcontroller/VCC_3V3
- U33 pad 5: Net-(U33-VOUT) -> +3V3
- U4 pad 10: unconnected-(U4-OUTS-Pad10) -> VDDA
- U8 pad 3: Net-(U8-3V3) -> /Microcontroller/VCC_3V3
- U8 pad 4: /GPIO0 -> /Microcontroller/GPIO0
- U8 pad 45: /CHIP_PU -> /Microcontroller/CHIP_PU
- U9 pad 2: CS_ -> /Ignition/CS_
- U9 pad 4: CS_ -> /Ignition/SDI
Routing:
- net /Vbias_AMP: track 30.9 -> 0.00 mm, vias 4 -> 0
- net /Insturmentation/Vbias: track 29.9 -> 1.51 mm
- net (no net): track 0.00 -> 28.4 mm
- net /SHIELD_AMP: track 20.7 -> 0.00 mm
- net VSSA: track 24.8 -> 7.38 mm, vias 4 -> 2
- net />PORE_AMP: track 14.8 -> 0.00 mm, vias 1 -> 0
- net VDDA: track 26.5 -> 12.9 mm
- net Net-(C1-Pad1): track 11.8 -> 0.00 mm
- net /Insturmentation/SHIELD: track 12.4 -> 3.53 mm
- net Net-(U14-S1): track 8.50 -> 0.00 mm
- net Net-(U14-S3): track 8.31 -> 0.00 mm
- net /GUARD: track 8.11 -> 0.00 mm
- net Net-(U3-+): track 0.00 -> 8.06 mm
- net Net-(J1-Pin_1): track 7.68 -> 0.00 mm
- net Net-(J2-Pin_1): track 7.03 -> 0.00 mm
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- removed copper zone on F.Cu, net GNDA
Other:
- board outline removed

Commit message: Signed-off-by: lokimetasmith <lokimail@gmail.com>
Parts:
- removed R130, R143: 27, Resistor_SMD:R_0402_1005Metric
- added C24: 4.7u, Capacitor_SMD:C_0402_1005Metric, F.Cu at (89.1, 37.6)
- added C26: 4.7u, Capacitor_SMD:C_0402_1005Metric, F.Cu at (89.1, 35.6)
- added R10: 27, Resistor_SMD:R_0402_1005Metric, F.Cu at (90.7, 66.1)
- added R13: 10k 1%, Resistor_SMD:R_0402_1005Metric, F.Cu at (77.9, 59.8)
- added R22: 10k 1%, Resistor_SMD:R_0402_1005Metric, F.Cu at (80.0, 59.8)
- added R27: 27, Resistor_SMD:R_0402_1005Metric, F.Cu at (85.3, 45.4)
- added R28: 27, Resistor_SMD:R_0402_1005Metric, F.Cu at (90.7, 62.8)
- added R33: 27, Resistor_SMD:R_0402_1005Metric, F.Cu at (90.7, 64.0)
- added R36: 27, Resistor_SMD:R_0402_1005Metric, F.Cu at (90.7, 65.0)
- added R37: 27, Resistor_SMD:R_0402_1005Metric, F.Cu at (90.7, 67.3)
- added R39: 27, Resistor_SMD:R_0402_1005Metric, F.Cu at (90.7, 68.4)
- added R40: 27, Resistor_SMD:R_0402_1005Metric, F.Cu at (90.7, 69.6)
- added R41: 27, Resistor_SMD:R_0402_1005Metric, F.Cu at (85.3, 43.4)
- added R42: 27, Resistor_SMD:R_0402_1005Metric, F.Cu at (89.0, 39.6)
- added R44: 1K, Resistor_SMD:R_0402_1005Metric, F.Cu at (85.3, 39.4)
- added R45: 1K, Resistor_SMD:R_0402_1005Metric, F.Cu at (85.3, 37.4)
- added R46: 1K, Resistor_SMD:R_0402_1005Metric, F.Cu at (85.3, 35.5)
- added U10: AD40xxBRMZ, Package_SO:MSOP-10_3x3mm_P0.5mm, F.Cu at (96.2, 38.3)
- added U6: ADA4940-1xCP, Package_CSP:LFCSP-16-1EP_3x3mm_P0.5mm_EP1.3x1.3mm_ThermalVias, F.Cu at (94.2, 44.0)
- R43: value 27 -> 1K
- U16: value LTC6268xS8-10 -> LTC6268xS8
- U3: footprint Package_SO:SOIC-8_3.9x4.9mm_P1.27mm -> Package_SO:VSSOP-8_3x3mm_P0.65mm
- moved C25 123.5 mm to (88.8, 28.8)
- moved C27 122.4 mm to (88.2, 31.9)
- moved R7 103.7 mm to (85.7, 74.4), turned to 180 degrees
- moved R20 103.5 mm to (82.8, 78.0), turned to 90 degrees
- moved R43 100.4 mm to (85.3, 41.4), turned to 180 degrees
- moved C18 99.9 mm to (79.5, 80.8), turned to -90 degrees
- moved R38 98.1 mm to (110.0, 86.8)
- moved C28 98.1 mm to (110.0, 88.8)
- moved C121 95.8 mm to (87.0, 55.8), turned to 0 degrees
- moved U4 93.7 mm to (73.1, 78.1), turned to 90 degrees
- moved U33 93.0 mm to (87.5, 61.9), turned to 90 degrees
- moved C119 92.2 mm to (90.2, 58.6), turned to 90 degrees
- moved R26 91.5 mm to (79.4, 75.3), turned to 90 degrees
- moved R19 91.3 mm to (73.0, 81.5), turned to -90 degrees
- moved R145 91.2 mm to (85.6, 65.0), turned to 0 degrees
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Connections:
- J12 pad 3: /Insturmentation/Vbias -> unconnected-(J12-Pin_3-Pad3)
- NT1 pad 1: +3.3V -> +3V3
- R35 pad 1: Net-(U13-OUT) -> Net-(R22-Pad1)
- R43 pad 1: /Microcontroller/GPIO40 -> GNDA
- R43 pad 2: /Microcontroller/TMUX_A0 -> Net-(U6A--IN)
- U1 pad 12: Net-(U1-EN+) -> unconnected-(U1-EN+-Pad12)
- U1 pad 8: Net-(U1-EN+) -> unconnected-(U1-EN--Pad8)
- U3 pad 1: unconnected-(U3-NC-Pad1) -> /Ignition/>PORE
- U3 pad 5: unconnected-(U3-NC-Pad5) -> GNDA
- U3 pad 6: /Ignition/>PORE -> Net-(U3B--)
- U3 pad 7: VDDA -> Net-(C26-Pad2)
- U3 pad 8: unconnected-(U3-NC-Pad8) -> VDDA
Routing:
- net (no net): track 28.4 -> 0.00 mm
- net +3V3: track 0.00 -> 22.9 mm
- net /Insturmentation/SHIELD: track 3.53 -> 23.8 mm
- net VBUS: track 3.65 -> 23.4 mm, vias 0 -> 1
- net /Ignition/CS_: track 0.00 -> 14.2 mm, vias 0 -> 2
- net /Ignition/SCK: track 0.00 -> 13.7 mm, vias 0 -> 2
- net VDDA: track 12.9 -> 26.0 mm
- net /Ignition/SDI: track 0.00 -> 12.4 mm, vias 0 -> 2
- net /Power/V_USB: track 14.1 -> 25.8 mm
- net /Ignition/LDAC_: track 0.00 -> 10.7 mm, vias 0 -> 2
- net /Power/-VIOC: track 0.00 -> 8.68 mm, vias 0 -> 1
- net /Insturmentation/Vbias: track 1.51 -> 9.70 mm, vias 1 -> 0
- net /Power/FB+: track 5.16 -> 12.8 mm, vias 0 -> 2
- net /Power/+Vp: track 5.83 -> 13.2 mm
- net VSSA: track 7.38 -> 14.2 mm
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Other:
- board outline added: 80 x 60 mm

Commit message: Signed-off-by: lokimetasmith <lokimail@gmail.com>
Parts:
- added C31: 100nF, Capacitor_SMD:C_0402_1005Metric, F.Cu at (79.1, 93.0)
- added C32: 100nF, Capacitor_SMD:C_0402_1005Metric, F.Cu at (79.1, 94.9)
- added C33: 100nF, Capacitor_SMD:C_0402_1005Metric, F.Cu at (79.1, 96.9)
- added C34: 100nF, Capacitor_SMD:C_0402_1005Metric, F.Cu at (86.4, 96.7)
- added C35: 10u, Capacitor_SMD:C_0402_1005Metric, F.Cu at (91.7, 34.2)
- added H2: MountingHole_Pad, MountingHole:MountingHole_6mm_Pad_Via, F.Cu at (62.4, 52.8)
- added H3: MountingHole_Pad, MountingHole:MountingHole_6mm_Pad_Via, F.Cu at (89.1, 52.2)
- added H4: MountingHole_Pad, MountingHole:MountingHole_6mm_Pad_Via, F.Cu at (62.4, 70.7)
- added H5: MountingHole_Pad, MountingHole:MountingHole_6mm_Pad_Via, F.Cu at (48.3, 66.0)
- added H6: MountingHole_Pad, MountingHole:MountingHole_3.2mm_M3_Pad_Via, F.Cu at (108.6, 35.5)
- added H7: MountingHole_Pad, MountingHole:MountingHole_3.2mm_M3_Pad_Via, F.Cu at (38.4, 35.5)
- added H8: MountingHole_Pad, MountingHole:MountingHole_3.2mm_M3_Pad_Via, F.Cu at (38.6, 85.2)
- added H9: MountingHole_Pad, MountingHole:MountingHole_3.2mm_M3_Pad_Via, F.Cu at (108.7, 85.5)
- added U11: LP5907MFX-1.8, Package_TO_SOT_SMD:SOT-23-5, F.Cu at (83.8, 97.3)
- moved R45 10.1 mm to (75.9, 33.7)
- moved C23 9.37 mm to (82.1, 82.0), turned to 180 degrees
- moved R34 9.09 mm to (115.5, 51.7)
- moved R7 7.54 mm to (82.1, 81.0), turned to 0 degrees
- moved R96 7.06 mm to (113.4, 56.8)
- moved R97 7.06 mm to (113.4, 55.8)
- moved R44 6.93 mm to (82.3, 33.1)
- moved J23 6.83 mm to (110.8, 44.0)
- moved C9 6.13 mm to (112.2, 51.1)
- moved J36 5.98 mm to (102.8, 45.1)
- moved R9 5.96 mm to (110.8, 51.1)
- moved C22 4.52 mm to (83.2, 79.8), turned to 0 degrees
- moved U8 4.43 mm to (104.1, 61.0)
- moved U10 4.06 mm to (98.5, 34.9), turned to 0 degrees
- moved C14 3.00 mm to (80.4, 80.8), turned to -90 degrees
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Connections:
- U10 pad 2: VDDA -> +1V8
Routing:
- net +3V3: track 22.9 -> 9.79 mm
- net /Ignition/CS_: track 14.2 -> 6.23 mm
- net /Ignition/SCK: track 13.7 -> 5.96 mm
- net VBUS: track 23.4 -> 15.9 mm
- net /Ignition/SDI: track 12.4 -> 5.18 mm
- net /Power/-VIOC: track 8.68 -> 2.77 mm, vias 1 -> 0
- net /Ignition/LDAC_: track 10.7 -> 5.83 mm
- net /Microcontroller/GPIO11: track 0.00 -> 2.58 mm
- net /Microcontroller/GPIO4: track 2.58 -> 0.00 mm
- net /Microcontroller/GPIO40: track 1.85 -> 0.00 mm
- net /Microcontroller/GPIO45: track 0.00 -> 1.76 mm
- net /Microcontroller/GPIO41: track 1.76 -> 0.00 mm
- net /Power/-Vp: track 19.3 -> 21.0 mm, vias 0 -> 1
- net /Microcontroller/TX: track 1.78 -> 0.18 mm
- net /Power/FB-: track 5.28 -> 4.26 mm
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