File: MR1/MR1.kicad_pcb (KiCad board)
At the start: 6 copper layers, 80 x 60 mm, 111 parts, among them J12 Conn_01x10, J22 B4B_PH, J23 Jumper_1, J3 USB_C_Receptacle_USB2.0, J36 Conn_ARM_JTAG_SWD_10, U1 LM27762, U10 AD40xxBRMZ, U11 LP5907MFX-1.8, U13 ADR4550, U16 LTC6268xS8, U3 OPA197xD, U33 NCP163ASN330T1G, U4 LT3045xDD, U5 LT3094xDD, U6 ADA4940-1xCP, U7 SN65220, U8 ESP32-S3-MINI-1U, U9 MCP4822, Y2 32.768 kHz

Commit message: commiting pcb changes
Parts:
- removed C19, C20, C34: 100nF, Capacitor_SMD:C_0402_1005Metric
- removed C35: 10u, Capacitor_SMD:C_0402_1005Metric
- removed H2, H3, H4, H5: MountingHole_Pad, MountingHole:MountingHole_6mm_Pad_Via
- removed J12: Conn_01x10, Connector_JST:JST_SH_SM10B-SRSS-TB_1x10-1MP_P1.00mm_Horizontal
- removed R27: 27, Resistor_SMD:R_0402_1005Metric
- removed R3, R43, R44, R45, R46, R5: 1K, Resistor_SMD:R_0402_1005Metric
- removed R4: 100, Resistor_SMD:R_0402_1005Metric
- removed U10: AD40xxBRMZ, Package_SO:MSOP-10_3x3mm_P0.5mm
- removed U11: LP5907MFX-1.8, Package_TO_SOT_SMD:SOT-23-5
- removed U16: LTC6268xS8, Package_SO:SO-8_3.9x4.9mm_P1.27mm
- removed U6: ADA4940-1xCP, Package_CSP:LFCSP-16-1EP_3x3mm_P0.5mm_EP1.3x1.3mm_ThermalVias
- added C36: 2pF, Capacitor_SMD:C_0402_1005Metric, F.Cu at (104.2, 82.2)
- added C37: 4.7u, Capacitor_SMD:C_0402_1005Metric, F.Cu at (65.8, 52.8)
- added C39: 100nF, Capacitor_SMD:C_0402_1005Metric, F.Cu at (70.5, 51.0)
- added C43: 1nF, Capacitor_SMD:C_0402_1005Metric, F.Cu at (64.4, 51.3)
- added D1: 1N4148WS, Diode_SMD:D_SOD-323, F.Cu at (47.4, 78.6)
- added D2: 1N4148WS, Diode_SMD:D_SOD-323, F.Cu at (59.3, 77.8)
- added J7: Conn_01x14_MountingPin, Connector_FFC-FPC:Amphenol_F32R-1A7x1-11014_1x14-1MP_P0.5mm_Horizontal, F.Cu at (75.8, 56.5)
- added Q1: 2SA1037, Package_TO_SOT_SMD:SOT-23, F.Cu at (58.9, 74.9)
- added Q2: CMBT2222A, Package_TO_SOT_SMD:SOT-23, F.Cu at (50.6, 78.4)
- added R47: 1M, Resistor_SMD:R_0402_1005Metric, F.Cu at (103.2, 82.2)
- added R48: 15K, Resistor_SMD:R_0402_1005Metric, F.Cu at (100.1, 74.6)
- added R52: 15K, Resistor_SMD:R_0402_1005Metric, F.Cu at (102.0, 74.5)
- added R53: 27, Resistor_SMD:R_0402_1005Metric, F.Cu at (100.1, 68.6)
- added R54: 27, Resistor_SMD:R_0402_1005Metric, F.Cu at (102.1, 68.6)
- added R55: 10k 1%, Resistor_SMD:R_0402_1005Metric, F.Cu at (99.1, 68.6)
- added R56: 10k 1%, Resistor_SMD:R_0402_1005Metric, F.Cu at (103.1, 68.6)
- added U12: SN65220, Package_TO_SOT_SMD:SOT-23-6, F.Cu at (101.0, 71.9)
- R21: value 82k 1% -> 1M
- R29: value 10k 1% -> 24k
- R31: value 3K9 -> 10k
- R35: value 3K9 -> 20k
- U13: value ADR4550 -> ADR4520
- moved C28 66.5 mm to (43.8, 83.1)
- moved R38 66.2 mm to (43.9, 84.2)
- moved C32 42.4 mm to (65.8, 54.6), turned to -90 degrees
- moved C33 38.1 mm to (70.9, 59.7), turned to 90 degrees
- moved C31 36.7 mm to (67.8, 58.0), turned to -90 degrees
- moved C25 36.6 mm to (66.7, 58.0), turned to -90 degrees
- moved C24 35.5 mm to (61.6, 60.0), turned to 90 degrees
- moved C26 34.7 mm to (64.1, 59.7), turned to 0 degrees
- moved C27 33.1 mm to (61.9, 52.0)
- moved R42 32.5 mm to (64.7, 61.2), turned to -90 degrees
- moved R41 21.3 mm to (86.1, 64.7), turned to 0 degrees
- moved U13 20.8 mm to (56.7, 55.2), turned to 180 degrees
- moved C23 19.1 mm to (64.9, 73.7), turned to 90 degrees
- moved C12 17.7 mm to (61.9, 51.0)
- moved R7 17.7 mm to (66.0, 73.7), turned to -90 degrees
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Connections:
- C14 pad 1: /Power/-Vp -> /Power/-Vp_cm
- C14 pad 2: GNDA -> GND
- C15 pad 1: GNDA -> GND
- C15 pad 2: /Power/+Vp -> /Power/+Vp_cm
- C16 pad 2: GNDA -> GND
- C18 pad 2: GNDA -> GND
- J3 pad A8: unconnected-(J3-SBU1-PadA8) -> /Power/SBU1
- J3 pad B8: unconnected-(J3-SBU2-PadB8) -> /Power/SBU2
- J36 pad 2: /Microcontroller/JTAG_TMS -> /Microcontroller/GPIO42
- J36 pad 4: /Microcontroller/JTAG_TCK -> /Microcontroller/GPIO39
- J36 pad 6: /Microcontroller/JTAG_TDO -> /Microcontroller/GPIO40
- J36 pad 8: /Microcontroller/JTAG_TDI -> /Microcontroller/GPIO41
- NT4 pad 1: /Insturmentation/Vbias -> Net-(C39-Pad1)
- R10 pad 1: /Ignition/SCK -> /Insturmentation/ADC_SDO
- R18 pad 1: /Power/-Vp -> /Power/-Vp_cm
- R21 pad 1: Net-(U3A-+) -> Net-(U3A--)
- R24 pad 2: /Power/+Vp -> /Power/+Vp_cm
- R25 pad 1: GNDA -> GND
- R26 pad 2: GNDA -> GND
- R28 pad 1: /Insturmentation/DAC_EN -> /Ignition/SCK
- R29 pad 2: Net-(U3A-+) -> Net-(U3A--)
- R31 pad 2: Net-(U3A-+) -> Net-(U3A--)
- R33 pad 1: /Ignition/LDAC_ -> /Insturmentation/ADC_SDI
- R35 pad 2: Net-(U3A-+) -> Net-(U3A--)
- R36 pad 1: /Ignition/CS_ -> /Insturmentation/ADC_EN
- R37 pad 1: /Ignition/SDI -> /Insturmentation/ADC_CLK
- R39 pad 1: /Microcontroller/DAC_Dout -> /Ignition/LDAC_
- R40 pad 1: /Insturmentation/DAC_CLK -> /Ignition/SDI
- R41 pad 1: Net-(U6A--OUT) -> /Ignition/CS_
- R41 pad 2: Net-(U10-IN-) -> /Microcontroller/GPIO12
- U1 pad 11: /Power/+Vp -> /Power/+Vp_cm
- U1 pad 13: GNDA -> GND
- U1 pad 4: GNDA -> GND
- U1 pad 6: /Power/-Vp -> /Power/-Vp_cm
- U3 pad 2: GNDA -> Net-(U3A--)
- U3 pad 3: Net-(U3A-+) -> GNDA
Routing:
- net VSSA: track 14.2 -> 57.9 mm, vias 2 -> 0
- net Earth: track 0.00 -> 27.6 mm
- net /Insturmentation/SHIELD: track 23.8 -> 0.00 mm, vias 2 -> 0
- net GND: track 13.4 -> 35.7 mm, vias 2 -> 6
- net /Power/SBU2: track 0.00 -> 20.5 mm, vias 0 -> 2
- net GNDA: track 27.2 -> 45.5 mm, vias 9 -> 8
- net VBUS: track 15.9 -> 31.2 mm, vias 1 -> 2
- net /Power/-Vp: track 21.0 -> 6.16 mm, vias 1 -> 0
- net /Insturmentation/ADC_CLK: track 0.00 -> 13.4 mm
- net /Insturmentation/ADC_SDO: track 0.00 -> 13.3 mm
- net /Insturmentation/ADC_SDI: track 0.00 -> 13.2 mm
- net /Insturmentation/ADC_EN: track 0.00 -> 13.0 mm
- net /Microcontroller/GPIO47: track 0.00 -> 12.4 mm
- net /Ignition/LDAC_: track 5.83 -> 17.7 mm, vias 2 -> 0
- net /Microcontroller/GPIO46: track 0.00 -> 11.3 mm, vias 0 -> 1
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- added copper zone on In2.Cu, net +3V3
- added copper zone on B.Cu, net GND
- added copper zone on F.Cu, net GND
- added copper zone on B.Cu, net GNDA
- added copper zone on F.Cu, net GNDA
Other:
- copper layers 6 -> 4

Commit message: updated board, and worked to improve the project, added .agents which might be a mistake, along with the board updates
Parts:
- added C40: 100u, Capacitor_SMD:C_1206_3216Metric, F.Cu at (76.9, 86.9)
- added C42: 100u, Capacitor_SMD:C_1206_3216Metric, F.Cu at (81.0, 74.0)
- added E1: SparkGap, Jumper:SolderJumper-2_P1.3mm_Open_TrianglePad1.0x1.5mm, F.Cu at (46.5, 88.3)
- added E2: SparkGap, Jumper:SolderJumper-2_P1.3mm_Open_TrianglePad1.0x1.5mm, F.Cu at (86.6, 87.9)
- U4: footprint Package_DFN_QFN:DFN-12-1EP_3x3mm_P0.5mm_EP1.6x2.5mm -> Package_DFN_QFN:DFN-12-1EP_3x3mm_P0.45mm_EP1.65x2.38mm_ThermalVias
- moved D1 27.2 mm to (73.7, 85.7), turned to 90 degrees
- moved Q2 26.5 mm to (76.5, 84.0), turned to 180 degrees
- moved Q1 18.8 mm to (77.7, 75.8), turned to 0 degrees
- moved D2 15.5 mm to (74.8, 76.8), turned to 90 degrees
- moved C32 7.25 mm to (70.0, 60.6)
- moved C37 7.20 mm to (70.0, 58.6)
- moved R24 6.56 mm to (80.3, 83.5)
- moved U13 5.90 mm to (61.3, 59.0)
- moved C10 5.78 mm to (86.4, 74.0)
- moved C118 5.78 mm to (86.4, 72.7)
- moved C119 5.78 mm to (85.7, 57.4)
- moved C121 5.78 mm to (83.7, 56.9)
- moved C13 5.78 mm to (75.1, 80.5)
- moved C14 5.78 mm to (80.8, 77.0)
- moved C16 5.78 mm to (80.5, 79.9)
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Connections:
- J22 pad 1: /Microcontroller/VCC_3V3 -> +3V3
- J22 pad 2: /Microcontroller/GPIO17 -> /Microcontroller/GPIO33
- J36 pad 1: /Microcontroller/VCC_3V3 -> +3V3
- R34 pad 1: /Microcontroller/VCC_3V3 -> +3V3
- R9 pad 1: /Microcontroller/VCC_3V3 -> +3V3
Routing:
- net VDDA: track 25.0 -> 44.2 mm, vias 0 -> 2
- net GNDA: track 45.5 -> 27.2 mm, vias 8 -> 12
- net VSSA: track 57.9 -> 44.1 mm, vias 0 -> 2
- net /Power/+Vp: track 10.6 -> 21.9 mm
- net /Microcontroller/GPIO33: track 0.00 -> 10.8 mm
- net Net-(U3A--): track 6.47 -> 16.2 mm, vias 1 -> 2
- net +3V3: track 13.9 -> 21.3 mm, vias 5 -> 8
- net /Power/-Vp: track 6.16 -> 11.7 mm
- net Net-(D2-A): track 0.00 -> 5.40 mm
- net /Power/+Vp_cm: track 6.05 -> 11.4 mm
- net Net-(D1-K): track 0.00 -> 4.69 mm
- net /Power/-VIOC: track 8.55 -> 13.1 mm
- net Earth: track 27.6 -> 23.1 mm
- net /Ignition/>PORE: track 11.6 -> 8.65 mm
- net GND: track 35.7 -> 38.5 mm, vias 6 -> 11
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- added copper zone on B.Cu, net Earth
- added copper zone on F.Cu, net Earth
- added copper zone on In1.Cu, net Earth
- added copper zone on In2.Cu, net Earth
- added copper zone on In1.Cu, net GND
- added copper zone on In1.Cu, net GNDA
- added copper zone on In2.Cu, net GNDA

Commit message: lots of refinements.
Parts:
- removed C37: 4.7u, Capacitor_SMD:C_0402_1005Metric
- removed U5: LT3094xDD, Package_DFN_QFN:DFN-12-1EP_3x3mm_P0.45mm_EP1.65x2.38mm_ThermalVias
- added C29: 100nF, Capacitor_SMD:C_0402_1005Metric, F.Cu at (70.4, 57.1)
- added R27: 27, Resistor_SMD:R_0402_1005Metric, F.Cu at (86.2, 65.1)
- added R43: 27, Resistor_SMD:R_0402_1005Metric, F.Cu at (70.5, 58.4)
- added U2: LT3094xDD, Package_DFN_QFN:DFN-12-1EP_3x3mm_P0.45mm_EP1.65x2.38mm_ThermalVias, F.Cu at (70.2, 78.8)
- D1, D2: value 1N4148WS -> 1N4148WT-7; footprint Diode_SMD:D_SOD-323 -> Diode_SMD:D_SOD-523
- U4: footprint Package_DFN_QFN:DFN-12-1EP_3x3mm_P0.45mm_EP1.65x2.38mm_ThermalVias -> Package_DFN_QFN:DFN-12-1EP_3x3mm_P0.5mm_EP1.6x2.5mm
- moved D2 1.73 mm to (76.0, 75.7)
- moved C42 1.10 mm to (81.0, 73.0)
- moved Q1 1.05 mm to (78.8, 75.8)
- moved R10 0.81 mm to (86.2, 64.1)
- moved R33 0.75 mm to (86.2, 62.0)
- moved R36 0.71 mm to (86.2, 63.0)
- moved NT2 0.50 mm to (71.5, 64.0)
- moved C33 0.47 mm to (71.4, 65.5), turned to 180 degrees
- moved D1 0.16 mm to (73.8, 85.7)
- moved R37 0.05 mm to (86.2, 66.1)
Connections:
- C14 pad 2: GND -> GNDA
- C15 pad 1: GND -> GNDA
- C16 pad 2: GND -> GNDA
- C18 pad 2: GND -> GNDA
- C26 pad 1: Net-(U3B--) -> Net-(U13-OUT)
- C40 pad 2: GND -> GNDA
- C42 pad 1: GND -> GNDA
- C43 pad 2: /Ignition/>PORE -> Net-(C43-Pad2)
- J7 pad 4: GND -> /Insturmentation/ROUTE_SEL
- R10 pad 2: /Microcontroller/GPIO7 -> /Microcontroller/GPIO6
- R29 pad 1: /Ignition/>PORE -> Net-(C43-Pad2)
- R33 pad 2: /Microcontroller/GPIO5 -> /Microcontroller/GPIO4
- R36 pad 2: /Microcontroller/GPIO6 -> /Microcontroller/GPIO5
- U1 pad 13: GND -> GNDA
- U1 pad 4: GND -> GNDA
- U3 pad 1: /Ignition/>PORE -> Net-(C43-Pad2)
- U4 pad 11: GNDA -> VDDA
- U4 pad 13: (no net) -> GNDA
Routing:
- net /Power/-VIOC: track 13.1 -> 0.00 mm
- net /Insturmentation/ROUTE_SEL: track 0.00 -> 12.8 mm
- net GND: track 38.5 -> 28.8 mm, vias 11 -> 30
- net Net-(C43-Pad2): track 0.00 -> 5.10 mm
- net /Ignition/>PORE: track 8.65 -> 3.77 mm
- net Net-(U3B--): track 5.64 -> 2.82 mm
- net /Microcontroller/GPIO4: track 0.00 -> 2.40 mm
- net +3V3: track 21.3 -> 19.1 mm
- net VDDA: track 44.2 -> 45.8 mm, vias 2 -> 3
- net GNDA: track 27.2 -> 25.7 mm, vias 12 -> 19
- net /Power/-Vp: track 11.7 -> 13.2 mm
- net /Insturmentation/SHIELD: track 0.00 -> 1.25 mm
- net VSSA: track 44.1 -> 43.0 mm
- net /Microcontroller/GPIO21: track 5.08 -> 6.08 mm
- net Net-(U13-OUT): track 9.65 -> 8.86 mm
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- added copper zone on In2.Cu, net GND
