File: MR1/Ignition.kicad_sch (KiCad schematic)
At the start: 0 parts

Commit message: Signed-off-by: lokimetasmith <lokimail@gmail.com>
Parts:
- added C11, C12: 10nF, Capacitor_SMD:C_0402_1005Metric, symbol Device:C
- added C25, C27: 100nF, Capacitor_SMD:C_0402_1005Metric, symbol Device:C
- added R21: 82k 1%, Resistor_SMD:R_0402_1005Metric, symbol Device:R_Small_US
- added R29: 10k 1%, Resistor_SMD:R_0402_1005Metric, symbol Device:R_Small_US
- added R31, R35: 3K9, Resistor_SMD:R_0402_1005Metric, symbol Device:R
- added U13: ADR4550, Package_SO:SOIC-8_3.9x4.9mm_P1.27mm, symbol Reference_Voltage:ADR4550
- added U3: OPA197xD, Package_SO:SOIC-8_3.9x4.9mm_P1.27mm, symbol Amplifier_Operational:OPA197xD
- added U9: MCP4822, Package_SO:SOIC-8-1EP_3.9x4.9mm_P1.27mm_EP2.29x3mm, symbol Analog_DAC:MCP4822
Connections:
- new net: R21.1, R29.2, R31.2, R35.2, U3.3 (+)
- new net: R35.1, U13.6 (OUT)
- new net: R31.1, U9.8 (VA)
- new net: R21.2, U9.6 (VB)
- new net +3V3: U9.1 (Vdd)
- new net >PORE: R29.1, U3.6
- new net CS_: U9.2 (~{CS})
- new net GNDA: C11.2, C12.2, C25.2, C27.2, U13.4 (GND), U3.2 (-), U9.7 (Vss)
- new net LDAC_: U9.5 (~{LDAC})
- new net SCK: U9.3 (SCK)
- new net SDI: U9.4 (SDI)
- new net VDDA: C11.1, C25.1, U13.2 (IN), U3.7 (V+)
- new net VSSA: C12.1, C27.1, U3.4 (V-)
Other:
- note added: "-1.024V"
- note added: "-2.4V to 2.4V"
- note added: "0V to 2.048V"
- note added: "0V to 250mV"
- note added: "C2 and C3 X5R"
- note added: "OPA197. It's JFET input stage, low offset voltage, and rail-to-rail outputs are compelling selling points."
- note added: "This is a solid core strategy, using precise reference voltages and a low-noise summing inverter to generate a stable, precise, bidirectional bias potential. However, the user's primary engineering objective—monitoring the minuscule, bidirectional picoampere currents essential for accurate nanopore designs—cannot be achieved with this schematic as drawn. The current summing inverters operate as l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"
- note added: "use a precision reference here"

Commit message: Signed-off-by: lokimetasmith <lokimail@gmail.com>
Parts:
- added C24, C26: 4.7u, Capacitor_SMD:C_0402_1005Metric, symbol Device:C_Small
- added R13, R22: 10k 1%, Resistor_SMD:R_0402_1005Metric, symbol Device:R_Small_US
- added R42: 27, Resistor_SMD:R_0402_1005Metric, symbol Device:R_Small_US
- added unit 3 of U3
- added unit 1 of U3
- U3: footprint Package_SO:SOIC-8_3.9x4.9mm_P1.27mm -> Package_SO:VSSOP-8_3x3mm_P0.65mm; symbol Amplifier_Operational:OPA197xD -> Amplifier_Operational:OPA2156xDGK
Connections:
- net >PORE: now also U3.1; no longer U3.6
- net GNDA: now also U3.5 (+), C24.2, U3.2 (-); no longer U3.2 (-)
- net VDDA: now also U3.8 (V+); no longer U3.7 (V+)
- net VSSA: now also U3.4 (V-); no longer U3.4 (V-)
- net at R21.1, R29.2, R31.2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: now also U3.3 (+); no longer U3.3 (+)
- net at U13.6 (OUT): now also R13.2; no longer R35.1
- new net: C24.1, C26.1, R13.1, R22.2, U3.6 (-)
- new net: R22.1, R35.1, R42.2
- new net: C26.2, R42.1, U3.7
Other:
- moved on the sheet: R29, R35, U13

Commit message: Signed-off-by: lokimetasmith <lokimail@gmail.com>
Parts:
- added C37, C38: 4.7u, Capacitor_SMD:C_0402_1005Metric, symbol Device:C_Small
- U13: value ADR4550 -> ADR4520; MPN (none) -> ADR4520ARZ-R7; Mouser PN (none) -> 584-ADR4520ARZ-R7; price (none) -> $6.16
- U3: MPN (none) -> OPA197IDGKT; Mouser PN (none) -> 595-OPA197IDGKT; price (none) -> $1.53
- U9: MPN (none) -> MCP4822T-E/SN; Mouser PN (none) -> 579-MCP4822TESN; price (none) -> $3.92
Connections:
- net >PORE: now also C37.1
- net GNDA: now also C37.2, C38.2
- net at R21.1, R29.2, R31.2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: now also C38.1
Other:
- note added: "ADR4520"
- moved on the sheet: R21, R31
