File: MR1/Ignition.kicad_sch (KiCad schematic)
At the start: 18 parts, among them U13 ADR4520, U3 OPA197xD, U9 MCP4822

Commit message: Signed-off-by: lokimetasmith <lokimail@gmail.com>
Parts:
- removed C38: 4.7u, Capacitor_SMD:C_0402_1005Metric, symbol Device:C_Small
- added C43: 1nF, Capacitor_SMD:C_0402_1005Metric, symbol Device:C_Small
- R21: value 82k 1% -> 1M
- R29: value 10k 1% -> 24k
- R31: value 3K9 -> 10k
- R35: value 3K9 -> 20k
Connections:
- net >PORE: now also C43.2
- net GNDA: now also U3.3 (+); no longer U3.2 (-)
- net at R21.1, R29.2, R31.2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: now also U3.2 (-), C43.1; no longer U3.3 (+)

Commit message: chore: prepare repository and documentation for open-source release
- Removed internal .agents scaffolding and updated .gitignore
- Added CONTRIBUTING.md with CAD, PCB, firmware, and PR guidelines
- Added CODE_OF_CONDUCT.md (Contributor Covenant v2.1)
- Added SECURITY.md with hardware safety and vulnerability disclosure policies
- Added CITATION.cff for academic and scientific publications
- Added Pump_firmware/README.md for STM32G431 subsystem
- Expanded BOM.md with mechanical, fluidic, PCB, and active electronics
- Updated README.md test badges, architecture, and documentation index
- Cleared hardcoded absolute developer paths in export_manager.py and KiCad files
- Fixed formatting in install.sh and metadata in package.json
Parts:
- removed C37: 4.7u, Capacitor_SMD:C_0402_1005Metric, symbol Device:C_Small
- added C29: 100nF, Capacitor_SMD:C_0402_1005Metric, symbol Device:C
- added R43: 27, Resistor_SMD:R_0402_1005Metric, symbol Device:R_Small_US
Connections:
- net >PORE: now also C29.1, R43.2; no longer C43.2, R29.1, U3.1
- net GNDA: now also C29.2
- net at C24.1, R13.1, R22.2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: no longer C26.1
- net at R13.2, U13.6 (OUT): now also C26.1
- new net: C43.2, R29.1, R43.1, U3.1
Other:
- moved on the sheet: R22

Commit message: lots of refinements.
Other:
- moved on the sheet: C29
Changed lines of the file:
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@@
 	(wire
 		(pts
-			(xy 138.43 83.82) (xy 138.43 85.09)
+			(xy 138.43 85.09) (xy 138.43 86.36)
 		)
 		(stroke
@@
 	(wire
 		(pts
-			(xy 138.43 74.93) (xy 138.43 76.2)
+			(xy 138.43 74.93) (xy 138.43 77.47)
 		)
 		(stroke
@@
 	(symbol
 		(lib_id "power:GNDA")
-		(at 138.43 85.09 0)
+		(at 138.43 86.36 0)
 		(unit 1)
 		(body_style 1)
@@
 		(fields_autoplaced yes)
 		(property "Reference" "#PWR0116"
-			(at 138.43 91.44 0)
+			(at 138.43 92.71 0)
 			(hide yes)
 			(show_name no)
@@
 		)
 		(property "Value" "GNDA"
-			(at 138.43 90.805 0)
+			(at 138.43 92.075 0)
 			(show_name no)
 			(do_not_autoplace no)
@@
 		)
 		(property "Footprint" ""
-			(at 138.43 85.09 0)
+			(at 138.43 86.36 0)
 			(hide yes)
 			(show_name no)
@@
 		)
 		(property "Datasheet" ""
-			(at 138.43 85.09 0)
+			(at 138.43 86.36 0)
 			(hide yes)
 			(show_name no)
@@
 		)
 		(property "Description" "Power symbol creates a global label with name \"GNDA\" , analog ground"
-			(at 138.43 85.09 0)
+			(at 138.43 86.36 0)
 			(hide yes)
 			(show_name no)
@@
 	(symbol
 		(lib_id "Device:C")
-		(at 138.43 80.01 0)
+		(at 138.43 81.28 0)
 		(unit 1)
 		(body_style 1)
@@
 		(dnp no)
 		(property "Reference" "C29"
-			(at 141.351 78.8416 0)
+			(at 141.351 80.1116 0)
 			(show_name no)
 			(do_not_autoplace no)
@@
 		)
 		(property "Value" "100nF"
-			(at 141.351 81.153 0)
+			(at 141.351 82.423 0)
 			(show_name no)
 			(do_not_autoplace no)
@@
 		)
 		(property "Footprint" "Capacitor_SMD:C_0402_1005Metric"
-			(at 139.3952 83.82 0)
+			(at 139.3952 85.09 0)
 			(hide yes)
 			(show_name no)
@@
 		)
 		(property "Datasheet" ""
-			(at 138.43 80.01 0)
+			(at 138.43 81.28 0)
 			(hide yes)
 			(show_name no)
@@
 		)
 		(property "Description" ""
-			(at 138.43 80.01 0)
+			(at 138.43 81.28 0)
 			(show_name no)
 			(do_not_autoplace no)
@@
 		)
 		(property "Mouser PN" ""
-			(at 138.43 80.01 0)
+			(at 138.43 81.28 0)
 			(hide yes)
 			(show_name no)

Commit message: added opamp_signal_conditioning and more refined repo
Parts:
- C11, C12: LCSC (none) -> C1525
- C24, C26: LCSC (none) -> C19702
- C25, C27, C29: LCSC (none) -> C15255
- C43: LCSC (none) -> C1523
- R13, R22, R31: LCSC (none) -> C60490
- R21: LCSC (none) -> C25488
- R29: LCSC (none) -> C25324
- R35: LCSC (none) -> C25310
- R42, R43: LCSC (none) -> C25078
- U13: LCSC (none) -> C659578
- U3: LCSC (none) -> C133554
- U9: LCSC (none) -> C16040
Changed lines of the file:
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@@
 			)
 		)
+		(property "LCSC" "C15255"
+			(at 100.0252 113.03 0)
+			(hide yes)
+			(effects
+				(font
+					(size 1.27 1.27)
+				)
+			)
+		)
 		(property "Datasheet" ""
 			(at 99.06 109.22 0)
@@
 			)
 		)
+		(property "LCSC" "C60490"
+			(at 53.34 40.64 0)
+			(hide yes)
+			(effects
+				(font
+					(size 1.27 1.27)
+				)
+			)
+		)
 		(property "Datasheet" ""
 			(at 53.34 40.64 0)
@@
 			)
 		)
+		(property "LCSC" "C15255"
+			(at 110.1852 113.03 0)
+			(hide yes)
+			(effects
+				(font
+					(size 1.27 1.27)
+				)
+			)
+		)
 		(property "Datasheet" ""
 			(at 109.22 109.22 0)
@@
 			)
 		)
+		(property "LCSC" "C25324"
+			(at 115.57 43.18 0)
+			(hide yes)
+			(effects
+				(font
+					(size 1.27 1.27)
+				)
+			)
+		)
 		(property "Datasheet" ""
 			(at 115.57 43.18 0)
@@
 			)
 		)
+		(property "LCSC" "C1525"
+			(at 75.8952 113.03 0)
+			(hide yes)
+			(effects
+				(font
+					(size 1.27 1.27)
+				)
+			)
+		)
 		(property "Datasheet" ""
 			(at 74.93 109.22 0)
@@
 			)
 		)
+		(property "LCSC" "C25310"
+			(at 100.33 44.958 90)
+			(hide yes)
+			(effects
+				(font
+					(size 1.27 1.27)
+				)
+			)
+		)
 		(property "Datasheet" ""
 			(at 100.33 43.18 0)
@@
 			)
 		)
+		(property "LCSC" "C133554"
+			(at 78.74 43.18 0)
+			(hide yes)
+			(effects
+				(font
+					(size 1.27 1.27)
+				)
+			)
+		)
 		(property "Datasheet" "http://www.ti.com/lit/ds/symlink/opa2156.pdf"
 			(at 78.74 43.18 0)
@@
 			)
 		)
+		(property "LCSC" "C133554"
+			(at 154.94 95.25 0)
+			(hide yes)
+			(effects
+				(font
+					(size 1.27 1.27)
+				)
+			)
+		)
 		(property "Datasheet" "http://www.ti.com/lit/ds/symlink/opa2156.pdf"
 			(at 154.94 95.25 0)
@@
 			)
 		)
+		(property "LCSC" "C133554"
+			(at 116.84 74.93 0)
+			(hide yes)
+			(effects
+				(font
+					(size 1.27 1.27)
+				)
+			)
+		)
 		(property "Datasheet" "http://www.ti.com/lit/ds/symlink/opa2156.pdf"
 			(at 116.84 74.93 0)
@@
 			)
 		)
+		(property "LCSC" "C19702"
+			(at 59.69 45.72 0)
+			(hide yes)
+			(effects
+				(font
+					(size 1.27 1.27)
+				)
+			)
+		)
 		(property "Datasheet" ""
 			(at 59.69 45.72 0)
@@
 			)
 		)
+		(property "LCSC" "C659578"
+			(at 43.18 48.26 0)
+			(hide yes)
+			(effects
+				(font
+					(size 1.27 1.27)
+				)
+			)
+		)
 		(property "Datasheet" "https://www.analog.com/media/en/technical-documentation/data-sheets/ADR4520_4525_4530_4533_4540_4550.pdf"
 			(at 43.18 49.53 0)
@@
 			)
 		)
+		(property "LCSC" "C60490"
+			(at 82.55 74.168 90)
+			(hide yes)
+			(effects
+				(font
+					(size 1.27 1.27)
+				)
+			)
+		)
 		(property "Datasheet" ""
 			(at 82.55 72.39 0)
@@
 			)
 		)
+		(property "LCSC" "C25078"
+			(at 92.71 43.18 0)
+			(hide yes)
+			(effects
+				(font
+					(size 1.27 1.27)
+				)
+			)
+		)
 		(property "Datasheet" ""
 			(at 92.71 43.18 0)
@@
 			)
 		)
+		(property "LCSC" "C25488"
+			(at 88.9 80.01 0)
+			(hide yes)
+			(effects
+				(font
+					(size 1.27 1.27)
+				)
+			)
+		)
 		(property "Datasheet" ""
 			(at 88.9 80.01 0)
@@
 			)
 		)
+		(property "LCSC" "C25078"
+			(at 134.62 74.93 0)
+			(hide yes)
+			(effects
+				(font
+					(size 1.27 1.27)
+				)
+			)
+		)
 		(property "Datasheet" ""
 			(at 134.62 74.93 0)
@@
 			)
 		)
+		(property "LCSC" "C16040"
+			(at 73.66 82.55 0)
+			(hide yes)
+			(effects
+				(font
+					(size 1.27 1.27)
+				)
+			)
+		)
 		(property "Datasheet" "http://ww1.microchip.com/downloads/en/DeviceDoc/20002249B.pdf"
 			(at 73.66 82.55 0)
@@
 			)
 		)
+		(property "LCSC" "C19702"
+			(at 74.93 34.29 0)
+			(hide yes)
+			(effects
+				(font
+					(size 1.27 1.27)
+				)
+			)
+		)
 		(property "Datasheet" ""
 			(at 74.93 34.29 0)
@@
 			)
 		)
+		(property "LCSC" "C15255"
+			(at 139.3952 85.09 0)
+			(hide yes)
+			(effects
+				(font
+					(size 1.27 1.27)
+				)
+			)
+		)
 		(property "Datasheet" ""
 			(at 138.43 81.28 0)
@@
 			)
 		)
+		(property "LCSC" "C1523"
+			(at 115.57 34.29 0)
+			(hide yes)
+			(effects
+				(font
+					(size 1.27 1.27)
+				)
+			)
+		)
 		(property "Datasheet" ""
 			(at 115.57 34.29 0)
@@
 			)
 		)
+		(property "LCSC" "C60490"
+			(at 76.2 24.13 0)
+			(hide yes)
+			(effects
+				(font
+					(size 1.27 1.27)
+				)
+			)
+		)
 		(property "Datasheet" ""
 			(at 76.2 24.13 0)
@@
 			(effects
 				(font
+					(size 1.27 1.27)
+				)
+			)
+		)
+		(property "LCSC" "C1525"
+			(at 88.5952 113.03 0)
+			(hide yes)
+			(effects
+				(font
