File: MR1/Insturmentation.kicad_sch (KiCad schematic)
At the start: 0 parts

Commit message: Signed-off-by: lokimetasmith <lokimail@gmail.com>
Parts:
- added C1: 2pF, Capacitor_SMD:C_0402_1005Metric, symbol Device:C
- added C19, C2, C20, C3, C6: 100nF, Capacitor_SMD:C_0402_1005Metric, symbol Device:C
- added C4, C5: 10nF, Capacitor_SMD:C_0402_1005Metric, symbol Device:C
- added H1: Nanopore, footprints:Nanopore holder_recessed, symbol Mechanical:MountingHole
- added J1, J10, J11, J2: Conn_01x01_Pin, footprints:Electrode, symbol Connector:Conn_01x01_Pin
- added J12, J9: Conn_01x10, Connector_JST:JST_SH_SM10B-SRSS-TB_1x10-1MP_P1.00mm_Horizontal, symbol MR1:Conn_01x11_MP
- added NT3, NT4: NetTie_2, NetTie:NetTie-2_SMD_Pad0.5mm, symbol Device:NetTie_2
- added R1: 1M, Resistor_SMD:R_0402_1005Metric, symbol Device:R
- added R3, R5, R6: 1K, Resistor_SMD:R_0402_1005Metric, symbol Device:R
- added R4, R8: 100, Resistor_SMD:R_0402_1005Metric, symbol Device:R
- added U16: LTC6268xS8-10, Package_SO:SO-8_3.9x4.9mm_P1.27mm, symbol MR1:LTC6268xS8-10_SHIELD
- added U2: LMP7721, Package_SO:SOIC-8_3.9x4.9mm_P1.27mm, symbol LMP7721:LMP7721
- added U6: MCP3301, symbol Analog_ADC:MCP3301
Connections:
- new net: C1.1, R1.1, R8.2, U2.4
- new net: C1.2, J1.1 (Pin_1), R1.2, U2.8 (-)
- new net: R3.1, U16.6, U6.2 (IN+)
- new net: R3.2, R4.2, U16.2 (-)
- new net: J2.1 (Pin_1), R6.2
- new net >PORE: J12.1 (Pin_1)
- new net >PORE_AMP: J10.1 (Pin_1), J9.1 (Pin_1)
- new net DAC_CLK: U6.7 (CLK)
- new net DAC_Dout: U6.6 (Dout)
- new net DAC_EN: U6.5 (~{CS}/SHDN)
- new net GNDA: C19.2, C2.2, C20.2, C3.2, C4.2, C5.2, C6.2, J12.2 (Pin_2), J12.6 (Pin_6), J9.2 (Pin_2), J9.6 (Pin_6), R5.2, U6.3 (IN-)
- new net GUARD: NT3.1, U2.2 (NC), U2.7 (NC)
- new net SHIELD: J12.10 (Pin_10), J12.4 (Pin_4), J12.9 (Pin_9), J12.MP (Pin_11), NT4.2
- new net SHIELD_AMP: J9.10 (Pin_10), J9.4 (Pin_4), J9.9 (Pin_9), J9.MP (Pin_11)
- new net Signal_AMP: J9.5 (Pin_5), R8.1
- new net Signal_Return: J12.5 (Pin_5), R5.1, U16.3 (+)
- new net VDDA: C19.1, C2.1, C4.1, J12.8 (Pin_8), J9.7 (Pin_7), U16.7 (V+), U2.6 (V+), U6.8 (Vdd)
- new net VSSA: C20.1, C3.1, C5.1, J12.7 (Pin_7), J9.8 (Pin_8), U16.5 (V-), U2.3 (V-), U6.4 (Vss)
- new net Vbias: J12.3 (Pin_3), NT4.1, R4.1, U16.1 (NC), U16.4 (NC), U6.1 (Vref)
- new net Vbias_AMP: C6.1, J11.1 (Pin_1), J9.3 (Pin_3), NT3.2, R6.1, U2.1 (+)
Other:
- note added: "250ft 32AWG CAT7 STP Solid, 0.075" Super Flat Bulk Ethernet Bare Copper Cable - White."
- note added: "3. Selecting the Precision ADC To capture <1µV signals, you need a 24-bit or 32-bit Delta-Sigma ADC. The standard 12-bit or 16-bit SAR ADCs used in microcontrollers will not see the signal floor you have created. Top Recommendations: TI ADS1261 (24-bit / 32-bit mode): Why: It has a built-in PGA (Programmable Gain Amplifier) that is extremely low noise. Noise Floor: Can resolve down to ~6 nV RMS a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"
- note added: "499Ω Metal Film Resistor"
- note added: "C2 and C3 X5R"
- note added: "LTC6268"
- note added: "LTC6268, alternate to TI's opamp"
- note added: "MCP33131"
- note added: "MG Chemicals 422C conformal coating"
- note added: "No, the schematic recipe I provided above is **Fixed Gain (10x)**. It uses a standard resistor, so the zoom level is locked. Since you are removing the MAX9939 (which *was* a variable gain amplifier), you likely want to keep that functionality—especially since Nanopores vary wildly in current. A 1 nA pore needs different gain than a 100 pA pore. Here is how to build a **"Safe" Variable Gain Ampli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"
- note added: "P1"
- note added: "P2"
- note added: "P3"
- note added: "P4"
- note added: "PGA855"
- note added: "PTFE (ZYF255DA): Dk .approx 2.55"
- note added: "R1 1206"
- note added: "SHR-10V-S"
- note added: "SM10B-SRSS-TB"
- note added: "SSH-003T-P0.2-H #32 to #28 (0.032 to 0.081) 0.4 to 0.8 23,000"
- note added: "Stage 1: Transimpedance Amp"
- note added: "Virtual Ground"
- note added: "amplifier board"
- note added: "consider cat 7 flat ribbon cable, 8 pairs, shielded"
- note added: "https://www.vpi.us/bulk-cable-sf/super-flat-cat7-736#idTab9"
- note added: "low noise voltage converters"
- note added: "pins for holding the board in place while applying adhesive https://www.mcmaster.com/98378A208/"

Commit message: Signed-off-by: lokimetasmith <lokimail@gmail.com>
Parts:
- removed U6: MCP3301, symbol Analog_ADC:MCP3301
- added C29, C30: 10nF, Capacitor_SMD:C_0402_1005Metric, symbol Device:C
- added R27, R41: 27, Resistor_SMD:R_0402_1005Metric, symbol Device:R_Small_US
- added R43, R44, R45, R46: 1K, Resistor_SMD:R_0402_1005Metric, symbol Device:R
- added U10: AD40xxBRMZ, Package_SO:MSOP-10_3x3mm_P0.5mm, symbol Analog_ADC:AD40xxBRMZ
- added U6: ADA4940-1xCP, Package_CSP:LFCSP-16-1EP_3x3mm_P0.5mm_EP1.3x1.3mm_ThermalVias, symbol Amplifier_Difference:ADA4940-1xCP
- U16: value LTC6268xS8-10 -> LTC6268xS8
Connections:
- net DAC_CLK: now also U10.8 (SCK)
- net DAC_EN: now also U10.6 (CNV)
- net GNDA: now also C29.1, C30.2, R43.1, U10.5 (GND), U6.17 (EP), U6.9 (VOCM)
- net VDDA: now also U10.2 (VDD), U6.5 (+Vs), U6.6 (+Vs), U6.7 (+Vs), U6.8 (+Vs)
- net VSSA: now also U6.13 (-Vs), U6.14 (-Vs), U6.15 (-Vs), U6.16 (-Vs)
- net Vbias: now also U10.1 (REF); no longer J12.3 (Pin_3)
- net at R3.1, U16.6: now also R45.1
- new net: C30.1, R41.2, U10.4 (IN-)
- new net: C29.2, R27.2, U10.3 (IN+)
- new net: R41.1, U6.11 (-OUT)
- new net: R27.1, U6.10 (+OUT)
- new net: R46.1, U6.1 (-FB)
- new net: R45.2, R46.2, U6.2 (+IN)
- new net: R43.2, R44.1, U6.3 (-IN)
- new net: R44.2, U6.4 (+FB)
- new net +3V3: U10.10 (VIO)
- new net DAC_SDI: U10.9 (SDI)
- new net DAC_SDO: U10.7 (SDO)
Other:
- note added: "Stage 2 Voltage Amplifier"

Commit message: Signed-off-by: lokimetasmith <lokimail@gmail.com>
Parts:
- added C31, C32, C33: 100nF, Capacitor_SMD:C_0402_1005Metric, symbol Device:C
- added C35: 10u, Capacitor_SMD:C_0402_1005Metric, symbol Device:C_Small
- U10: MPN (none) -> AD4011BCPZ-RL7; Mouser PN (none) -> 584-AD4011BCPZ-RL7; price (none) -> $21.70
- U16: MPN (none) -> LTC6268IS8#TRPBF; Mouser PN (none) -> 584-LTC6268IS8#TRPBF; price (none) -> $8.40
- U2: MPN (none) -> LMP7721MA/NOPB; price (none) -> $5.13
- U6: MPN (none) -> ADA4940-1ACPZ-RL; Mouser PN (none) -> 584-ADA4940-1ACPZ-R; price (none) -> $4.57
Connections:
- net +3V3: now also C33.1
- net GNDA: now also C31.2, C32.2, C33.2, C35.2
- net VDDA: now also C31.1; no longer U10.2 (VDD)
- net VSSA: now also C32.1
- net Vbias: now also C35.1
- new net +1V8: U10.2 (VDD)

Commit message: Signed-off-by: lokimetasmith <lokimail@gmail.com>
Parts:
- added C39: 100nF, Capacitor_SMD:C_0402_1005Metric, symbol Device:C
Connections:
- net GNDA: now also C39.2
- net Vbias: no longer NT4.1
- new net: C39.1, NT4.1
Other:
- note added: "RF-damping capacitor"
