File: MR1/Microcontroller.kicad_sch (KiCad schematic)
At the start: 0 parts

Commit message: Signed-off-by: lokimetasmith <lokimail@gmail.com>
Parts:
- added C119, C7: 10u, Capacitor_SMD:C_0402_1005Metric, symbol Device:C_Small
- added C51, C52: 12p, Capacitor_SMD:C_0402_1005Metric, symbol Device:C_Small
- added C9: 4.7u, Capacitor_SMD:C_0402_1005Metric, symbol Device:C_Small
- added J22: B4B_PH, Connector_JST:JST_PH_B4B-PH-K_1x04_P2.00mm_Vertical, symbol Connector_Generic:Conn_01x04
- added J23: Jumper_1, Connector_PinHeader_2.54mm:PinHeader_1x02_P2.54mm_Vertical, symbol Connector:Conn_01x02_Pin
- added J36: Conn_ARM_JTAG_SWD_10, Connector_PinHeader_1.27mm:PinHeader_2x05_P1.27mm_Vertical_SMD, symbol Connector:Conn_ARM_JTAG_SWD_10
- added NT1: NetTie_2, NetTie:NetTie-2_SMD_Pad0.5mm, symbol Device:NetTie_2
- added R130, R143, R43, R96, R97: 27, Resistor_SMD:R_0402_1005Metric, symbol Device:R_Small_US
- added R30: 1M, Resistor_SMD:R_0402_1005Metric, symbol Device:R_Small_US
- added R32, R51: 0, Resistor_SMD:R_0402_1005Metric, symbol Device:R_Small_US
- added R34, R9: 10k 1%, Resistor_SMD:R_0402_1005Metric, symbol Device:R_Small_US
- added SW1, SW2: SW_Push, Custom Footprints:SW_SPST_6mm_gull wing, symbol Switch:SW_Push
- added TP11: TestPoint, TestPoint:TestPoint_Pad_D1.0mm, symbol Connector:TestPoint
- added U8: ESP32-S3-MINI-1U, RF_Module:ESP32-S2-MINI-1U, symbol RF_Module:ESP32-S3-MINI-1U
- added Y2: 32.768 kHz, Crystal:Crystal_SMD_3215-2Pin_3.2x1.5mm, symbol Device:Crystal
Connections:
- new net: C51.2, R30.1, R32.1, Y2.2
- new net: C52.2, R30.2, R51.2, Y2.1
- new net +3.3V: NT1.1
- new net CHIP_PU: C9.1, J36.10 (~{RESET}), R9.2, SW2.2, U8.45 (EN)
- new net GND: C119.2, C51.1, C52.1, C7.2, C9.2, J22.4 (Pin_4), J23.1 (Pin_1), J36.3 (GND), J36.5 (GND), J36.9 (GNDDetect), SW1.1, SW2.1, U8.1 (GND), U8.2 (GND), U8.42 (GND), U8.43 (GND), U8.46 (GND), U8.47 (GND), U8.48 (GND), U8.49 (GND), U8.50 (GND), U8.51 (GND), U8.52 (GND), U8.53 (GND), U8.54 (GND), U8.55 (GND), U8.56 (GND), U8.57 (GND), U8.58 (GND), U8.59 (GND), U8.60 (GND), U8.61 (GND), U8.62 (GND), U8.63 (GND), U8.64 (GND), U8.65 (GND)
- new net GPIO0: R143.2, SW1.2, U8.4 (IO0)
- new net GPIO1: U8.5 (IO1)
- new net GPIO10: U8.14 (IO10)
- new net GPIO11: U8.15 (IO11)
- new net GPIO12: U8.16 (IO12)
- new net GPIO13: U8.17 (IO13)
- new net GPIO14: U8.18 (IO14)
- new net GPIO15: R32.2, U8.19 (IO15)
- new net GPIO16: R51.1, U8.20 (IO16)
- new net GPIO17: J22.2 (Pin_2), U8.21 (IO17)
- new net GPIO18: U8.22 (IO18)
- new net GPIO2: U8.6 (IO2)
- new net GPIO21: U8.25 (IO21)
- new net GPIO26: U8.26 (IO26)
- new net GPIO3: U8.7 (IO3)
- new net GPIO33: U8.28 (IO33)
- new net GPIO34: U8.29 (IO34)
- new net GPIO35: U8.31 (IO35)
- new net GPIO36: U8.32 (IO36)
- new net GPIO37: U8.33 (IO37)
- new net GPIO38: U8.34 (IO38)
- new net GPIO39: U8.35 (IO39)
- new net GPIO4: U8.8 (IO4)
- new net GPIO40: R43.1, U8.36 (IO40)
- new net GPIO41: R130.1, U8.37 (IO41)
- new net GPIO42: U8.38 (IO42)
- new net GPIO45: U8.41 (IO45)
- new net GPIO46: J23.2 (Pin_2), R34.2, U8.44 (IO46)
- new net GPIO47: J22.3 (Pin_3), U8.27 (IO47)
- new net GPIO48: U8.30 (IO48)
- new net GPIO5: U8.9 (IO5)
- new net GPIO6: U8.10 (IO6)
- new net GPIO7: U8.11 (IO7)
- new net GPIO8: U8.12 (IO8)
- new net GPIO9: U8.13 (IO9)
- new net JTAG_TCK: J36.4 (SWCLK/TCK)
- new net JTAG_TDI: J36.8 (NC/TDI)
- new net JTAG_TDO: J36.6 (SWO/TDO)
- new net JTAG_TMS: J36.2 (SWDIO/TMS)
- new net RX: R97.1, U8.40 (RXD0)
- new net RXD0: R96.2
- new net TMUX_A0: R43.2
- new net TMUX_A1: R130.2
- new net TX: R96.1, U8.39 (TXD0)
- new net TXD0: R97.2
- new net USB_D+: U8.24 (USB_D+)
- new net USB_D-: U8.23 (USB_D-)
- new net VCC_3V3: C119.1, C7.1, J22.1 (Pin_1), J36.1 (VTref), NT1.2, R34.1, R9.1, TP11.1, U8.3 (3V3)
Other:
- note added: "9.0PF"
- note added: "ADC1: 10 channels: GPIO1 - GPIO10 ADC2 is shared with WiFi"
- note added: "Boot Mode | GPIO0 | GPIO46 Default Config | 1(pull-up)| 0 (Pull-down) SPI Boot | 1 | Any Value Joint DL Boot | 0 | 0 Invalid | 0 | 1"
- note added: "Jumper"
- note added: "UART TTL or SPI, selectable in firmware"
- note added: "Y2: ESR = Max. 70 KΩ 32.768 kHz"

Commit message: Signed-off-by: lokimetasmith <lokimail@gmail.com>
Parts:
- removed R130, R143, R43: 27, Resistor_SMD:R_0402_1005Metric, symbol Device:R_Small_US
- added R10, R28, R33, R36, R37, R39, R40: 27, Resistor_SMD:R_0402_1005Metric, symbol Device:R_Small_US
Connections:
- net GPIO10: now also R40.2
- net GPIO11: now also R28.2
- net GPIO5: now also R33.2
- net GPIO6: now also R36.2
- net GPIO7: now also R10.2
- net GPIO8: now also R37.2
- net GPIO9: now also R39.2
- net +3.3V renamed +3V3
- new net CS_: R36.1
- new net DAC_CLK: R40.1
- new net DAC_Dout: R39.1
- new net DAC_EN: R28.1
- new net LDAC_: R33.1
- new net SCK: R10.1
- new net SDI: R37.1
Other:
- moved on the sheet: C51, C52, J22, R30, R32, R51, Y2

Commit message: Signed-off-by: lokimetasmith <lokimail@gmail.com>
Parts:
- U8: Mouser PN (none) -> 356-ESP32S3MINI1UN8; price (none) -> $5.50
- Y2: Mouser PN (none) -> 732-N32768K90NN60KC5; price (none) -> $0.431
Changed lines of the file:
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@@
 			)
 		)
+		(property "Mouser PN" "732-N32768K90NN60KC5"
+			(at 57.15 110.49 90)
+			(effects
+				(font
+					(size 1.27 1.27)
+				)
+				(hide yes)
+			)
+		)
+		(property "price" "$0.431	"
+			(at 57.15 110.49 90)
+			(effects
+				(font
+					(size 1.27 1.27)
+				)
+				(hide yes)
+			)
+		)
 		(pin "2"
 		)
@@
 			(at 195.58 68.58 0)
 			(effects
+				(font
+					(size 1.27 1.27)
+				)
+				(hide yes)
+			)
+		)
+		(property "Mouser PN" "356-ESP32S3MINI1UN8"
+			(at 195.58 68.58 0)
+			(effects
+				(font
+					(size 1.27 1.27)
+				)
+				(hide yes)
+			)
+		)
+		(property "price" "$5.50	"
+			(at 195.58 68.58 0)
+			(effects
