File: MR1/Microcontroller.kicad_sch (KiCad schematic)
At the start: 28 parts, among them J22 B4B_PH, J23 Jumper_1, J36 Conn_ARM_JTAG_SWD_10, SW1 SW_Push, SW2 SW_Push, U8 ESP32-S3-MINI-1U, Y2 32.768 kHz

Commit message: Signed-off-by: lokimetasmith <lokimail@gmail.com>
Changed lines of the file:
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@@
 	(wire
 		(pts
+			(xy 170.18 148.59) (xy 168.91 148.59)
+		)
+		(stroke
+			(width 0)
+			(type default)
+		)
+	)
+	(wire
+		(pts
 			(xy 49.53 104.14) (xy 57.15 104.14)
 		)
@@
 	(wire
 		(pts
-			(xy 168.91 147.32) (xy 168.91 149.86)
+			(xy 170.18 148.59) (xy 170.18 149.86)
 		)
 		(stroke
@@
 	(wire
 		(pts
+			(xy 165.1 148.59) (xy 166.37 148.59)
+		)
+		(stroke
+			(width 0)
+			(type default)
+		)
+	)
+	(wire
+		(pts
+			(xy 166.37 148.59) (xy 166.37 147.32)
+		)
+		(stroke
+			(width 0)
+			(type default)
+		)
+	)
+	(wire
+		(pts
 			(xy 154.94 53.34) (xy 180.34 53.34)
 		)
@@
 	(wire
 		(pts
+			(xy 168.91 148.59) (xy 168.91 147.32)
+		)
+		(stroke
+			(width 0)
+			(type default)
+		)
+	)
+	(wire
+		(pts
 			(xy 210.82 66.04) (xy 238.76 66.04)
 		)
@@
 	(wire
 		(pts
-			(xy 166.37 147.32) (xy 166.37 149.86)
+			(xy 165.1 148.59) (xy 165.1 149.86)
 		)
 		(stroke
@@
 	(symbol
 		(lib_id "power:GND")
-		(at 168.91 149.86 0)
+		(at 170.18 149.86 0)
 		(unit 1)
 		(body_style 1)
@@
 		(fields_autoplaced yes)
 		(property "Reference" "#PWR0139"
-			(at 168.91 156.21 0)
+			(at 170.18 156.21 0)
 			(hide yes)
 			(show_name no)
@@
 		)
 		(property "Value" "GND"
-			(at 168.91 154.94 0)
+			(at 170.18 154.94 0)
 			(show_name no)
 			(do_not_autoplace no)
@@
 		)
 		(property "Footprint" ""
-			(at 168.91 149.86 0)
+			(at 170.18 149.86 0)
 			(hide yes)
 			(show_name no)
@@
 		)
 		(property "Datasheet" ""
-			(at 168.91 149.86 0)
+			(at 170.18 149.86 0)
 			(hide yes)
 			(show_name no)
@@
 		)
 		(property "Description" "Power symbol creates a global label with name \"GND\" , ground"
-			(at 168.91 149.86 0)
+			(at 170.18 149.86 0)
 			(hide yes)
 			(show_name no)
@@
 	(symbol
 		(lib_id "power:GND")
-		(at 166.37 149.86 0)
+		(at 165.1 149.86 0)
 		(unit 1)
 		(body_style 1)
@@
 		(fields_autoplaced yes)
 		(property "Reference" "#PWR0138"
-			(at 166.37 156.21 0)
+			(at 165.1 156.21 0)
 			(hide yes)
 			(show_name no)
@@
 		)
 		(property "Value" "GND"
-			(at 166.37 154.94 0)
+			(at 165.1 154.94 0)
 			(show_name no)
 			(do_not_autoplace no)
@@
 		)
 		(property "Footprint" ""
-			(at 166.37 149.86 0)
+			(at 165.1 149.86 0)
 			(hide yes)
 			(show_name no)
@@
 		)
 		(property "Datasheet" ""
-			(at 166.37 149.86 0)
+			(at 165.1 149.86 0)
 			(hide yes)
 			(show_name no)
@@
 		)
 		(property "Description" "Power symbol creates a global label with name \"GND\" , ground"
-			(at 166.37 149.86 0)
+			(at 165.1 149.86 0)
 			(hide yes)
 			(show_name no)

Commit message: feat(cad,firmware,interposer): PTFE interposer, deliverables pipeline, and firmware
- CAD & Interposer:
  - Modeled PTFE_Interposer (55.0 x 51.962 x 0.8 mm) with central wafer diamond cutout
  - Dual-sided silver chloride (Ag/AgCl) ribbon electrode pads (30 deg Cis, 210 deg Trans)
  - 6-pad pogo pin landing array and 4 fluidic pass-throughs with weep duct relief
  - Verified 0 physical collisions across cartridge stack and housings (100% green)
- Deliverables & Export Pipeline:
  - Created automated export system (Makefile, scripts/export_manager.py, scripts/export_all.sh)
  - Full cataloging of 159 deliverables (30 STLs, 13 DXFs, STEPs, Gerbers, WireViz)
  - Added E2E tests (tests/test_exports_e2e.py) and legacy parity tests (tests/test_legacy_feature_parity.py)
- Firmware & Schematics:
  - ESP32-S3 firmware with 100 kHz USB streaming, FreeRTOS dual-core tasks, Web UI
  - Added fast AD40xx SPI driver, MCP4822 DAC driver, leak detection, and pump UART
  - SBU auto-polarity detection and I2C routing in MR1 schematics
- Docs & Environment:
  - Added setup_env.sh, setup_env.ps1, requirements.txt, EXPORTS.md
  - Updated README.md, TODO.md, atlas.project.json, and walkthrough.md
Parts:
- added R55, R56: 10k 1%, Resistor_SMD:R_0402_1005Metric, symbol Device:R_Small_US
Connections:
- net +3V3: now also R55.1, R56.2
- net GPIO21 renamed USB_SCL
- net USB_SCL: now also R56.1
- net GPIO26 renamed USB_SDA
- net USB_SDA: now also R55.2
Other:
- note added: "sbu pins usb"

Commit message: commiting pcb changes
Parts:
- added R41: 27, Resistor_SMD:R_0402_1005Metric, symbol Device:R_Small_US
Connections:
- net DAC_CLK is gone; now on net SDI: R40.1
- net DAC_Dout is gone; now on net LDAC_: R39.1
- net DAC_EN is gone; now on net SCK: R28.1
- net JTAG_TCK is gone; now on net GPIO39: J36.4 (SWCLK/TCK)
- net JTAG_TDI is gone; now on net GPIO41: J36.8 (NC/TDI)
- net JTAG_TDO is gone; now on net GPIO40: J36.6 (SWO/TDO)
- net JTAG_TMS is gone; now on net GPIO42: J36.2 (SWDIO/TMS)
- net CS_: now also R41.1; no longer R36.1
- net GPIO12: now also R41.2
- net LDAC_: no longer R33.1
- net SCK: no longer R10.1
- net SDI: no longer R37.1
- net USB_SCL: now also U8.26 (IO26); no longer U8.25 (IO21)
- net USB_SDA: now also U8.25 (IO21); no longer U8.26 (IO26)
- new net ADC_CLK: R37.1
- new net ADC_EN: R36.1
- new net ADC_SDI: R33.1
- new net ADC_SDO: R10.1
Other:
- moved on the sheet: J22

Commit message: updated board, and worked to improve the project, added .agents which might be a mistake, along with the board updates
Connections:
- net +3V3: now also J22.1 (Pin_1), J36.1 (VTref), R34.1, R9.1
- net GPIO17: no longer J22.2 (Pin_2)
- net GPIO33: now also J22.2 (Pin_2)
- net VCC_3V3: no longer J22.1 (Pin_1), J36.1 (VTref), R34.1, R9.1
Other:
- moved on the sheet: C9, R9
