File: MR1/Microcontroller.kicad_sch (KiCad schematic)
At the start: 31 parts, among them J22 B4B_PH, J23 Jumper_1, J36 Conn_ARM_JTAG_SWD_10, SW1 SW_Push, SW2 SW_Push, U8 ESP32-S3-MINI-1U, Y2 32.768 kHz

Commit message: lots of refinements.
Parts:
- added R27: 27, Resistor_SMD:R_0402_1005Metric, symbol Device:R_Small_US
Connections:
- net GPIO4: now also R33.2
- net GPIO5: now also R36.2; no longer R33.2
- net GPIO6: now also R10.2; no longer R36.2
- net GPIO7: now also R27.2; no longer R10.2
- new net ROUTE_SEL: R27.1
Other:
- moved on the sheet: C9, R10, R33, R36, R9

Commit message: added opamp_signal_conditioning and more refined repo
Parts:
- C119, C7: LCSC C1713 -> C1713
- C51, C52: LCSC (none) -> C1550
- C9: LCSC (none) -> C19702
- J22: LCSC (none) -> C131334
- J23: LCSC (none) -> C492401
- J36: LCSC (none) -> C521634
- R10, R27, R28, R33, R36, R37, R39, R40, R41, R96, R97: LCSC (none) -> C25078
- R30: LCSC (none) -> C25488
- R32, R51: LCSC (none) -> C25740
- R34, R55, R56, R9: LCSC (none) -> C60490
- SW1, SW2: LCSC (none) -> C481177
- U8: LCSC (none) -> C2980299
- Y2: LCSC (none) -> C91275
