File: MR1/Power.kicad_sch (KiCad schematic)
At the start: 0 parts

Commit message: Signed-off-by: lokimetasmith <lokimail@gmail.com>
Parts:
- added C10, C13, C14, C15, C18, C23, C8: 4.7u, Capacitor_SMD:C_0402_1005Metric, symbol Device:C_Small
- added C118, C121, C16, C17: 10u, Capacitor_SMD:C_0402_1005Metric, symbol Device:C_Small
- added C21, C22: 22u, Capacitor_SMD:C_0402_1005Metric, symbol Device:C_Small
- added D82: MBR0540, Diode_SMD:D_SOD-123, symbol Diode:MBR0540
- added J3: USB_C_Receptacle_USB2.0, Connector_USB:USB_C_Receptacle_HRO_TYPE-C-31-M-12, symbol Connector:USB_C_Receptacle_USB2.0
- added NT2: NetTie_2, NetTie:NetTie-2_SMD_Pad0.5mm, symbol Device:NetTie_2
- added R11, R12: 15K, Resistor_SMD:R_0402_1005Metric, symbol temp-sensor-rescue:R_Small_US-Device-temp-sensor-rescue
- added R14, R17: 5.1k, Resistor_SMD:R_0402_1005Metric, symbol temp-sensor-rescue:R_Small_US-Device-temp-sensor-rescue
- added R145: 10k, Resistor_SMD:R_0402_1005Metric, symbol Device:R
- added R15, R16: 27, Resistor_SMD:R_0402_1005Metric, symbol temp-sensor-rescue:R_Small_US-Device-temp-sensor-rescue
- added R18, R23, R24, R25, R26: 10k 1%, Resistor_SMD:R_0402_1005Metric, symbol Device:R_Small_US
- added R19: 9.16k, Resistor_SMD:R_0402_1005Metric, symbol Device:R_Small_US
- added R2, R7: 24.9k 0.1%, Resistor_SMD:R_0402_1005Metric, symbol Device:R
- added R20: 9.09k, Resistor_SMD:R_0402_1005Metric, symbol Device:R_Small_US
- added U1: LM27762, Package_SON:WSON-12-1EP_3x2mm_P0.5mm_EP1x2.65_ThermalVias, symbol Regulator_SwitchedCapacitor:LM27762
- added U33: NCP163ASN330T1G, Package_TO_SOT_SMD:SOT-23-5, symbol Regulator_Linear:NCP163ASN330T1G
- added U4: LT3045xDD, Package_DFN_QFN:DFN-12-1EP_3x3mm_P0.5mm_EP1.6x2.5mm, symbol MR1:LT3045xDD-1
- added U5: LT3094xDD, Package_DFN_QFN:DFN-12-1EP_3x3mm_P0.45mm_EP1.65x2.38mm_ThermalVias, symbol Regulator_Linear:LT3094xDD
- added U7: SN65220, Package_TO_SOT_SMD:SOT-23-6, symbol twig:SN65220-Power_Protection_passthrough
Connections:
- new net: C23.2, R7.1, U5.8 (SET)
- new net: R145.2, U33.3 (EN)
- new net: R23.2, U1.1 (PGOOD)
- new net: C8.2, R2.1, U4.8 (SET)
- new net: C13.1, U1.10 (C+)
- new net: C13.2, U1.9 (C-)
- new net: C18.1, U1.5 (CP)
- new net: U1.12 (EN+), U1.8 (EN-)
- new net +3V3: C121.1, U33.5 (VOUT)
- new net +VIOC: R19.1, U4.3 (VIOC)
- new net +Vp: C15.2, R24.2, U1.11 (OUT+), U4.1 (IN), U4.2 (IN), U4.4 (EN/UV), U4.7 (PGFB)
- new net -VIOC: R20.1, U5.7 (VIOC)
- new net -Vp: C14.1, R18.1, U1.6 (OUT-), U5.1 (IN), U5.13 (IN), U5.2 (IN), U5.3 (EN/UV), U5.5 (PGFB)
- new net CC1: J3.A5 (CC1), R17.2
- new net CC2: J3.B5 (CC2), R14.2
- new net D+: J3.A6 (D+), J3.B6 (D+), R11.1, R15.1, U7.1, U7.6 (A)
- new net D-: J3.A7 (D-), J3.B7 (D-), R12.2, R16.1, U7.3, U7.4 (B)
- new net Earth: J3.S1 (SHIELD)
- new net FB+: R19.2, R24.1, R25.2, U1.2 (FB+)
- new net FB-: R18.2, R20.2, R26.1, U1.7 (FB-)
- new net GND: C10.2, C118.2, C121.2, C17.2, J3.A1 (GND), J3.A12 (GND), J3.B1 (GND), J3.B12 (GND), NT2.2, R11.2, R12.1, R14.1, R17.1, U33.2 (GND), U7.2 (GND), U7.5 (GND)
- new net GNDA: C14.2, C15.1, C16.2, C18.2, C21.1, C22.1, C23.1, C8.1, NT2.1, R2.2, R25.1, R26.2, R7.2, U1.13 (PAD), U1.4 (GND), U4.11 (OUT), U4.6 (ILIM), U4.9 (GND), U5.6 (ILIM), U5.9 (GND)
- new net USB_D+: R15.2
- new net USB_D-: R16.2
- new net VBUS: C10.1, C118.1, C16.1, C17.1, D82.1 (K), R145.1, R23.1, U1.3 (VIN), U33.1 (VIN)
- new net VDDA: C21.2, U4.10 (OUTS), U4.11 (OUT), U4.12 (OUT)
- new net VSSA: C22.2, U5.10 (OUTS), U5.11 (OUT), U5.12 (OUT)
- new net V_USB: D82.2 (A), J3.A4 (VBUS), J3.A9 (VBUS), J3.B4 (VBUS), J3.B9 (VBUS)
- no-connect marks 0 -> 2
Other:
- note added: "+VOUT = 1.2 V × (R1 + R2) / R2 -VOUT = -1.22 V × (R3 + R4) / R4"
- note added: "3045-1"
- note added: "ESD"
- note added: "TPS7A94"
- note added: "place R19 and R20 or place R18 and R24, not both."

Commit message: Signed-off-by: lokimetasmith <lokimail@gmail.com>
Connections:
- net at U1.12 (EN+): no longer U1.8 (EN-)
Changed lines of the file:
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@@
-	(wire
-		(pts
-			(xy 40.64 52.07) (xy 40.64 54.61)
-		)
-		(stroke
-			(width 0)
-			(type default)
-		)
-	)
 	(wire
 		(pts
@@
 	(wire
 		(pts
-			(xy 40.64 54.61) (xy 44.45 54.61)
-		)
-		(stroke
-			(width 0)
-			(type default)
-		)
-	)
-	(wire
-		(pts
 			(xy 129.54 170.18) (xy 119.38 170.18)
 		)
@@
 		)
 		(stroke
-			(width 0)
-			(type default)
-		)
-	)
-	(wire
-		(pts
-			(xy 44.45 52.07) (xy 40.64 52.07)
-		)
-		(stroke

Commit message: Signed-off-by: lokimetasmith <lokimail@gmail.com>
Parts:
- added C34: 100nF, Capacitor_SMD:C_0402_1005Metric, symbol Device:C
- added U11: LP5907MFX-1.8, Package_TO_SOT_SMD:SOT-23-5, symbol Regulator_Linear:LP5907MFX-1.8
- D82: MPN (none) -> MBR0540L-TP; Mouser PN (none) -> 833-MBR0540L-TP; price (none) -> $0.273
- U1: MPN (none) -> LM27762DSSR; Mouser PN (none) -> 595-LM27762DSSR; price (none) -> $1.52
- U33: MPN NCP163ASN330T1G -> NCP114ASN330T1G; Mouser PN (none) -> 863-NCP114ASN330T1G; price 1 -> $0.095
- U4: MPN (none) -> LT3045EDD-1#TRPBF; Mouser PN (none) -> 584-LT3045EDD-1TRPBF; price (none) -> $7.13
- U5: MPN (none) -> LT3094EDD#TRPBF; Mouser PN (none) -> 584-LT3094EDD#TRPBF; price (none) -> $7.13
- U7: MPN (none) -> SN65220DBVR; Mouser PN (none) -> 595-SN65220DBVR; price (none) -> $1.74
Connections:
- net GNDA: now also C34.2, U11.2 (GND)
- net VDDA: now also U11.1 (IN), U11.3 (EN)
- new net +1V8: C34.1, U11.5 (OUT)
