File: MR1/Power.kicad_sch (KiCad schematic)
At the start: 50 parts, among them J3 USB_C_Receptacle_USB2.0, Q1 2SA1037, Q2 CMBT2222A, U1 LM27762, U12 SN65220, U33 NCP163ASN330T1G, U4 LT3045xDD, U5 LT3094xDD, U7 SN65220

Commit message: lots of refinements.
Parts:
- removed U5: LT3094xDD, Package_DFN_QFN:DFN-12-1EP_3x3mm_P0.45mm_EP1.65x2.38mm_ThermalVias, symbol Regulator_Linear:LT3094xDD
- added U2: LT3094xDD, Package_DFN_QFN:DFN-12-1EP_3x3mm_P0.45mm_EP1.65x2.38mm_ThermalVias, symbol MR1:LT3094xDD
- D1, D2: value 1N4148WS -> 1N4148WT-7; footprint Diode_SMD:D_SOD-323 -> Diode_SMD:D_SOD-523
- U4: footprint Package_DFN_QFN:DFN-12-1EP_3x3mm_P0.45mm_EP1.65x2.38mm_ThermalVias -> Package_DFN_QFN:DFN-12-1EP_3x3mm_P0.5mm_EP1.6x2.5mm
Connections:
- net -VIOC: now also U2.7 (VIOC)
- net -Vp: now also U2.1 (IN), U2.13 (IN), U2.2 (IN), U2.3 (EN/UV), U2.5 (PGFB)
- net GND: no longer C14.2, C15.1, C16.2, C18.2, C40.2, C42.1, U1.13 (PAD), U1.4 (GND)
- net GNDA: now also C14.2, C15.1, C16.2, C18.2, C40.2, C42.1, U1.13 (PAD), U1.4 (GND), U4.13 (GND), U2.6 (ILIM), U2.9 (GND); no longer U4.11 (OUT)
- net VSSA: now also U2.10 (OUTS), U2.11 (OUT), U2.12 (OUT)
- net at C23.2, R7.1: now also U2.8 (SET)

Commit message: added opamp_signal_conditioning and more refined repo
Parts:
- C10, C13, C14, C15, C18, C23, C8: LCSC (none) -> C19702
- C118, C121: LCSC C1713 -> C1713
- C16, C17: LCSC (none) -> C1713
- C21, C22: LCSC C1713 -> C23737
- C40, C42: LCSC (none) -> C15008
- D1, D2: LCSC (none) -> C107849
- D82: LCSC (none) -> C5204747
- J3: LCSC (none) -> C165948
- Q1: LCSC (none) -> C14902
- Q2: LCSC (none) -> C2152
- R11, R12, R48, R52: LCSC (none) -> C25275
- R14, R17: LCSC (none) -> C25212
- R15, R16, R53, R54: LCSC (none) -> C25078
- R18, R23, R24, R25, R26: LCSC (none) -> C60490
- R19: LCSC (none) -> C25991
- R2, R7: LCSC (none) -> C25327
- R20: LCSC (none) -> C25879
- R49, R50: LCSC (none) -> C25149
- U1: LCSC (none) -> C473398
- U12, U7: LCSC (none) -> C21787
- U2: LCSC (none) -> C670493
- U4: LCSC (none) -> C514420
