File: MR1/amplifier.kicad_pcb (KiCad board)
At the start: 6 copper layers, 8.8 x 8.8 mm, 104 parts, among them J1 Conn_01x01_Pin, J10 Conn_01x01_Pin, J11 Conn_01x01_Pin, J12 Conn_01x10, J2 Conn_01x01_Pin, J22 B4B_PH, J23 Jumper_1, J3 USB_C_Receptacle_USB2.0, J36 Conn_ARM_JTAG_SWD_10, J9 Conn_01x10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

Commit message: Signed-off-by: lokimetasmith <lokimail@gmail.com>
Parts:
- removed C10, C13, C14, C15, C18, C23, C8, C9: 4.7u, Capacitor_SMD:C_0402_1005Metric
- removed C11, C12: 0.1u, Capacitor_SMD:C_0402_1005Metric
- removed C118, C119, C120, C121, C16, C17, C7: 10u, Capacitor_SMD:C_0402_1005Metric
- removed C19, C20: 100nF, Capacitor_SMD:C_0402_1005Metric
- removed C21, C22: 22u, Capacitor_SMD:C_0402_1005Metric
- removed C51, C52: 12p, Capacitor_SMD:C_0402_1005Metric
- removed D82: MBR0540, Diode_SMD:D_SOD-123
- removed J12: Conn_01x10, Connector_JST:JST_SH_SM10B-SRSS-TB_1x10-1MP_P1.00mm_Horizontal
- removed J22: B4B_PH, Connector_JST:JST_PH_B4B-PH-K_1x04_P2.00mm_Vertical
- removed J23: Jumper_1, Connector_PinHeader_2.54mm:PinHeader_1x02_P2.54mm_Vertical
- removed J3: USB_C_Receptacle_USB2.0, Connector_USB:USB_C_Receptacle_HRO_TYPE-C-31-M-12
- removed J36: Conn_ARM_JTAG_SWD_10, Connector_PinHeader_1.27mm:PinHeader_2x05_P1.27mm_Vertical_SMD
- removed NT1, NT2, NT4: NetTie_2, NetTie:NetTie-2_SMD_Pad0.5mm
- removed R10, R13, R27, R28, R3, R5: 1K, Resistor_SMD:R_0402_1005Metric
- removed R11, R12: 15K, Resistor_SMD:R_0402_1005Metric
- removed R130, R143, R15, R16, R43, R96, R97: 27, Resistor_SMD:R_0402_1005Metric
- removed R14, R17: 5.1k, Resistor_SMD:R_0402_1005Metric
- removed R145, R146: 10k, Resistor_SMD:R_0402_1005Metric
- removed R18, R21, R22, R23, R24, R25, R26, R29, R33, R34, R9: 10k 1%, Resistor_SMD:R_0402_1005Metric
- removed R19: 9.16k, Resistor_SMD:R_0402_1005Metric
- removed R2, R7: 24.9k 0.1%, Resistor_SMD:R_0402_1005Metric
- removed R20: 9.09k, Resistor_SMD:R_0402_1005Metric
- removed R30: 1M, Resistor_SMD:R_0402_1005Metric
- removed R31, R35, R40: 3K9, Resistor_SMD:R_0402_1005Metric
- removed R32, R51: 0, Resistor_SMD:R_0402_1005Metric
- removed R4: 100, Resistor_SMD:R_0402_1005Metric
- removed TP11: TestPoint, TestPoint:TestPoint_Pad_D1.0mm
- removed U1: LM27762, Package_SON:WSON-12-1EP_3x2mm_P0.5mm_EP1x2.65_ThermalVias
- removed U12, U13: ADR4550, Package_SO:SOIC-8_3.9x4.9mm_P1.27mm
- removed U14: TMUX1104dgsr, Package_SO:VSSOP-10_3x3mm_P0.5mm
- removed U16: LTC6268xS8-10, Package_SO:SO-8_3.9x4.9mm_P1.27mm
- removed U33, U34: NCP163ASN330T1G, Package_TO_SOT_SMD:SOT-23-5
- removed U4: LT3045xDD, Package_DFN_QFN:DFN-12-1EP_3x3mm_P0.5mm_EP1.6x2.5mm
- removed U5: LT3094xDD, Package_DFN_QFN:DFN-12-1EP_3x3mm_P0.45mm_EP1.65x2.38mm_ThermalVias
- removed U7: SN65220, Package_TO_SOT_SMD:SOT-23-6
- removed U8: ESP32-S3-MINI-1U, RF_Module:ESP32-S2-MINI-1U
- removed U9: MCP4822, Package_SO:SOIC-8-1EP_3.9x4.9mm_P1.27mm_EP2.29x3mm
- removed Y2: 32.768 kHz, Crystal:Crystal_SMD_3215-2Pin_3.2x1.5mm
- moved R1 0.31 mm to (169.4, 65.3)
- moved C1 0.27 mm to (168.9, 66.1)
Routing:
- net /Vbias: track 29.9 -> 0.00 mm, vias 1 -> 0
- net /-Vp: track 15.4 -> 0.00 mm
- net GNDA: track 33.0 -> 18.8 mm, vias 4 -> 0
- net /V_USB: track 14.1 -> 0.00 mm
- net VDDA: track 26.5 -> 13.7 mm, vias 2 -> 0
- net /SHIELD: track 12.4 -> 0.00 mm, vias 2 -> 0
- net /D-: track 12.4 -> 0.00 mm
- net GND: track 11.7 -> 0.00 mm
- net /D+: track 10.8 -> 0.00 mm
- net Net-(U6-IN+): track 9.19 -> 0.00 mm
- net Net-(U14-S1): track 8.50 -> 0.00 mm
- net Net-(U14-S3): track 8.31 -> 0.00 mm
- net VSSA: track 24.8 -> 17.4 mm, vias 4 -> 2
- net /Signal_Return: track 6.91 -> 0.00 mm
- net Net-(U14-S2): track 6.83 -> 0.00 mm
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Other:
- copper layers 6 -> 2
