File: Amplifier/Amplifier.kicad_sch (KiCad schematic)
At the start: 17 parts, among them J1 Conn_01x01_Pin, J10 Conn_01x01_Pin, J11 Conn_01x01_Pin, J2 Conn_01x01_Pin, J9 Conn_01x10, U2 LMP7721

Commit message: Signed-off-by: lokimetasmith <lokimail@gmail.com>
Parts:
- added C19: 100nF, Capacitor_SMD:C_0402_1005Metric, symbol Device:C
- added C20: 100nF, Capacitor_SMD:C_0805_2012Metric, symbol Device:C
- added NT4, NT5: NetTie_2, NetTie:NetTie-2_SMD_Pad0.5mm, symbol Device:NetTie_2
- added Q1: JFE2140D, Package_SO:SOIC-8_3.9x4.9mm_P1.27mm, symbol Transistor_FET:JFE2140D
- added Q2: Q_NJFET_DSG, symbol Device:Q_NJFET_DSG
- added R3, R5: 1K, Resistor_SMD:R_0805_2012Metric, symbol Device:R
- added R4: 100, Resistor_SMD:R_0402_1005Metric, symbol Device:R
- added R9: 100, Resistor_SMD:R_0805_2012Metric, symbol Device:R
- added U16: LTC6268xS8, Package_SO:SO-8_3.9x4.9mm_P1.27mm, symbol MR1:LTC6268xS8-10_SHIELD
- C2, C6: footprint Capacitor_SMD:C_0402_1005Metric -> Capacitor_SMD:C_0805_2012Metric
- J1, J10, J11, J2: footprint footprints:Electrode -> footprints:Electrode_Guard
- R8: footprint Resistor_SMD:R_0402_1005Metric -> Resistor_SMD:R_0805_2012Metric
Connections:
- net >PORE_AMP: now also J2.1 (Pin_1), J9.10 (Pin_10); no longer J10.1 (Pin_1), J9.1 (Pin_1)
- net GNDA: now also J10.1 (Pin_1), J9.8 (Pin_8), J9.9 (Pin_9), C19.2, C20.2, NT4.1, R5.2; no longer J9.2 (Pin_2)
- net SHIELD_AMP: now also J9.1 (Pin_1), J9.2 (Pin_2), NT4.2; no longer J9.10 (Pin_10), J9.4 (Pin_4), J9.9 (Pin_9)
- net Signal_AMP: now also J9.3 (Pin_3), R9.1; no longer J9.5 (Pin_5), R8.1
- net VDDA: now also J9.5 (Pin_5), C19.1, Q1.1, Q1.2, Q1.3 (VCH), U16.7 (V+); no longer J9.7 (Pin_7)
- net VSSA: now also J9.7 (Pin_7), C20.1, Q1.7 (VCL), Q1.8, U16.5 (V-); no longer J9.8 (Pin_8)
- net Vbias_AMP: now also J9.4 (Pin_4), NT5.2, Q2.1 (D), Q2.2 (S); no longer C6.1, J11.1 (Pin_1), J9.3 (Pin_3), NT3.2, R6.1, U2.1 (+)
- net at R6.2: now also J11.1 (Pin_1); no longer J2.1 (Pin_1)
- new net: R3.1, R9.2, U16.6
- new net: R3.2, R4.2, U16.2 (-)
- new net: R5.1, R8.1, U16.3 (+)
- new net: Q1.4, Q1.5, Q1.6
- new net Vbias: C6.1, NT3.2, NT5.1, R4.1, R6.1, U16.1 (NC), U16.4 (NC), U2.1 (+)
Other:
- removed sheet Ignition
- removed sheet Insturmentation
- removed sheet Microcontroller
- removed sheet Power
- note added: "Ceramic capacitors are piezoelectric – mechanical vibrations and noises will create charge across the capacitor. Be careful when using ceramic caps in the input, integration, feedback or biasing networks."
- note added: "LSK170D-SOT-23-3L-CT"
- note added: "LSK489-SOT-23-6L-CT"
- note added: "LTC6268"
- note added: "Stage 2 Voltage Amplifier"
- moved on the sheet: C1, C2, C3, C4, C5, C6, H1, J1, J10, J11, J2, J9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
