File: Amplifier/amplifier.kicad_pcb (KiCad board)
At the start: 2 copper layers, 55 x 52 mm, 17 parts, among them J1 Conn_01x01_Pin, J10 Conn_01x01_Pin, J11 Conn_01x01_Pin, J2 Conn_01x01_Pin, J9 Conn_01x10, U2 LMP7721

Commit message: Signed-off-by: lokimetasmith <lokimail@gmail.com>
Parts:
- added C19: 100nF, Capacitor_SMD:C_0402_1005Metric, F.Cu at (172.5, 67.9)
- added C20: 100nF, Capacitor_SMD:C_0805_2012Metric, F.Cu at (153.8, 71.5)
- added NT4: NetTie_2, NetTie:NetTie-2_SMD_Pad0.5mm, F.Cu at (158.4, 76.9)
- added NT5: NetTie_2, NetTie:NetTie-2_SMD_Pad0.5mm, F.Cu at (163.0, 76.8)
- added R3: 1K, Resistor_SMD:R_0805_2012Metric, F.Cu at (159.2, 68.6)
- added R4: 100, Resistor_SMD:R_0402_1005Metric, F.Cu at (161.4, 68.4)
- added R5: 1K, Resistor_SMD:R_0805_2012Metric, F.Cu at (165.0, 73.2)
- added R9: 100, Resistor_SMD:R_0805_2012Metric, F.Cu at (153.9, 73.5)
- added U16: LTC6268xS8, Package_SO:SO-8_3.9x4.9mm_P1.27mm, F.Cu at (159.4, 72.3)
- C2, C6: footprint Capacitor_SMD:C_0402_1005Metric -> Capacitor_SMD:C_0805_2012Metric
- J1, J2: footprint footprints:Electrode -> footprints:Electrode_Guard; moved to B.Cu
- J10, J11: footprint footprints:Electrode -> footprints:Electrode_Guard; moved to F.Cu
- R8: footprint Resistor_SMD:R_0402_1005Metric -> Resistor_SMD:R_0805_2012Metric
- moved C2 17.2 mm to (153.9, 75.4)
- moved R6 11.8 mm to (162.5, 64.9), turned to 180 degrees
- moved C5 8.02 mm to (166.9, 75.2), turned to 0 degrees
- moved C4 7.01 mm to (164.5, 75.4), turned to 0 degrees
- moved R8 3.31 mm to (165.0, 71.1), turned to 0 degrees
- moved C1 1.94 mm to (169.5, 64.0), turned to 0 degrees
- moved R1 1.91 mm to (169.5, 63.0), turned to 0 degrees
- moved C3 1.88 mm to (163.3, 68.3), turned to -90 degrees
- moved U2 1.76 mm to (167.5, 67.2), turned to 0 degrees
- moved C6 1.16 mm to (162.1, 66.3), turned to 180 degrees
- moved NT3 0.73 mm to (165.0, 66.0), turned to 90 degrees
- moved J9 0.51 mm to (164.6, 79.1)
- turned J1 to -30 degrees
- turned J10 to 30 degrees
- turned J11 to 30 degrees
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Connections:
- C6 pad 1: /Vbias_AMP -> /Vbias
- J10 pad 1: />PORE_AMP -> GNDA
- J11 pad 1: /Vbias_AMP -> Net-(J11-Pin_1)
- J2 pad 1: Net-(J2-Pin_1) -> />PORE_AMP
- J9 pad 1: />PORE_AMP -> /SHIELD_AMP
- J9 pad 10: /SHIELD_AMP -> />PORE_AMP
- J9 pad 2: GNDA -> /SHIELD_AMP
- J9 pad 3: /Vbias_AMP -> /Signal_AMP
- J9 pad 4: /SHIELD_AMP -> /Vbias_AMP
- J9 pad 5: /Signal_AMP -> VDDA
- J9 pad 7: VDDA -> VSSA
- J9 pad 8: VSSA -> GNDA
- J9 pad 9: /SHIELD_AMP -> GNDA
- NT3 pad 2: /Vbias_AMP -> /Vbias
- R6 pad 1: /Vbias_AMP -> /Vbias
- R6 pad 2: Net-(J2-Pin_1) -> Net-(J11-Pin_1)
- R8 pad 1: /Signal_AMP -> Net-(U16-+)
- U2 pad 1: /Vbias_AMP -> /Vbias
Routing:
- net /Vbias_AMP: track 39.8 -> 0.00 mm, vias 5 -> 0
- net /Vbias: track 0.00 -> 36.1 mm
- net VDDA: track 13.7 -> 29.6 mm, vias 0 -> 3
- net /Signal_AMP: track 1.87 -> 16.0 mm
- net GNDA: track 18.8 -> 6.26 mm, vias 0 -> 30
- net VSSA: track 17.8 -> 26.6 mm, vias 2 -> 3
- net Net-(U16--): track 0.00 -> 7.24 mm
- net Net-(J2-Pin_1): track 7.03 -> 0.00 mm
- net Net-(R3-Pad1): track 0.00 -> 6.84 mm
- net Net-(U16-+): track 0.00 -> 5.27 mm
- net Net-(J11-Pin_1): track 0.00 -> 5.08 mm, vias 0 -> 1
- net /GUARD: track 8.11 -> 3.45 mm
- net Net-(J1-Pin_1): track 7.68 -> 3.54 mm
- net /SHIELD_AMP: track 20.7 -> 18.2 mm
- net Net-(C1-Pad1): track 11.8 -> 10.7 mm
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- added copper zone on B.Cu, net GNDA
