File: Amplifier/amplifier.kicad_pcb (KiCad board)
At the start: 2 copper layers, 55 x 52 mm, 26 parts, among them J1 Conn_01x01_Pin, J10 Conn_01x01_Pin, J11 Conn_01x01_Pin, J2 Conn_01x01_Pin, J9 Conn_01x10, U16 LTC6268xS8, U2 LMP7721

Commit message: Signed-off-by: lokimetasmith <lokimail@gmail.com>
Parts:
- J1, J10, J11, J2: footprint footprints:Electrode_Guard -> footprints:Electrode_Guard_Shield
- moved J1 1.94 mm to (170.9, 61.1), turned to 150 degrees
Routing:
- net /GUARD: track 3.45 -> 9.74 mm, vias 0 -> 11
- net VSSA: track 26.6 -> 28.1 mm

Commit message: Signed-off-by: lokimetasmith <lokimail@gmail.com>
Parts:
- moved J2 1.92 mm to (178.6, 65.5), turned to 150 degrees
Routing:
- net /Vbias: track 36.1 -> 34.9 mm
Changed lines of the file:
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@@
 		(capping no)
 		(filling no)
-		(zone_defaults)
 		(pcbplotparams
 			(layerselection 0x00000000_00000000_55555555_5755f5ff)
@@
 	(footprint "footprints:Electrode_Guard_Shield"
 		(layer "B.Cu")
-		(at 177.63134 67.201025 -30)
+		(at 178.595144 65.541773 150)
 		(property "Reference" "J2"
-			(at 0 0.5 150)
+			(at 0 0.5 330)
 			(unlocked yes)
 			(layer "B.SilkS")
@@
 		)
 		(property "Value" "Conn_01x01_Pin"
-			(at 0 -2.6 150)
+			(at 0 -2.6 330)
 			(unlocked yes)
 			(layer "B.Fab")
@@
 		)
 		(property "Datasheet" ""
-			(at 0 0 150)
+			(at 0 0 330)
 			(unlocked yes)
 			(layer "B.Fab")
@@
 		)
 		(property "Description" "small coaxial connector (BNC, SMA, SMB, SMC, Cinch/RCA, LEMO, ...)"
-			(at 0 0 150)
+			(at 0 0 330)
 			(unlocked yes)
 			(layer "B.Fab")
@@
 		)
 		(property "Alternate Part Number 1" ""
-			(at 0 0 330)
+			(at 0 0 150)
 			(unlocked yes)
 			(layer "B.Fab")
@@
 		)
 		(property "AssemblyType" ""
-			(at 0 0 330)
+			(at 0 0 150)
 			(unlocked yes)
 			(layer "B.Fab")
@@
 		)
 		(property "Configuration" ""
-			(at 0 0 330)
+			(at 0 0 150)
 			(unlocked yes)
 			(layer "B.Fab")
@@
 		)
 		(property "Distributor 2 PN" ""
-			(at 0 0 330)
+			(at 0 0 150)
 			(unlocked yes)
 			(layer "B.Fab")
@@
 		)
 		(property "MPN" ""
-			(at 0 0 330)
+			(at 0 0 150)
 			(unlocked yes)
 			(layer "B.Fab")
@@
 		)
 		(property "Manufacturer" ""
-			(at 0 0 330)
+			(at 0 0 150)
 			(unlocked yes)
 			(layer "B.Fab")
@@
 		)
 		(property "Manufacturer_Name" ""
-			(at 0 0 330)
+			(at 0 0 150)
 			(unlocked yes)
 			(layer "B.Fab")
@@
 		)
 		(property "Manufacturer_Part_Number" ""
-			(at 0 0 330)
+			(at 0 0 150)
 			(unlocked yes)
 			(layer "B.Fab")
@@
 		)
 		(property "Mouser Part Number" ""
-			(at 0 0 330)
+			(at 0 0 150)
 			(unlocked yes)
 			(layer "B.Fab")
@@
 		)
 		(property "Mouser Price/Stock" ""
-			(at 0 0 330)
+			(at 0 0 150)
 			(unlocked yes)
 			(layer "B.Fab")
@@
 		)
 		(property "price" ""
-			(at 0 0 330)
+			(at 0 0 150)
 			(unlocked yes)
 			(layer "B.Fab")
@@
 		)
 		(fp_line
-			(start -1.24 -0.05)
-			(end 1.2 -0.05)
+			(start -1.25 -1.85)
+			(end 1.26 -1.85)
 			(stroke
 				(width 0.1)
@@
 		)
 		(fp_line
-			(start -1.25 -1.85)
-			(end 1.26 -1.85)
+			(start -1.24 -0.05)
+			(end 1.2 -0.05)
 			(stroke
 				(width 0.1)
@@
 		)
 		(fp_text user "${REFERENCE}"
-			(at 0 -4.03 150)
+			(at 0 -4.03 330)
 			(unlocked yes)
 			(layer "B.Fab")
@@
 		)
 		(pad "1" thru_hole circle
-			(at 0 -0.95 330)
+			(at 0 -0.95 150)
 			(size 0.7 0.7)
 			(drill 0.5)
@@
 		)
 		(pad "2" smd roundrect
-			(at -0.698842 -1.648841 330)
+			(at -0.698842 -1.648841 150)
 			(size 0.2 0.2)
 			(layers "F.Cu" "F.Mask")
@@
 		)
 		(pad "2" smd roundrect
-			(at 0.698841 -1.648841 330)
+			(at 0.698841 -1.648841 150)
 			(size 0.2 0.2)
 			(layers "F.Cu" "F.Mask")
@@
 		(layer "B.Mask")
 	)
-	(gr_poly
-		(pts
-			(xy 106.67 117.73) (xy 106.67 108.04) (xy 112.39 102.32) (xy 112.39 102.15) (xy 102.55 96.32) (xy 92.55 101.31)
-			(xy 92.44 117.59)
-		)
-		(stroke
-			(width 0.1)
-			(type solid)
-		)
-		(fill no)
-		(layer "Dwgs.User")
-	)
 	(gr_line
 		(start 136.9983 54.167084)
@@
 		(start 151.3332 75.072934)
 		(end 151.3332 76.454)
-		(width 0.2)
+		(width 0.35)
 		(layer "F.Cu")
 		(net "/Signal_AMP")
@@
 		(start 155.8354 76.9302)
 		(end 156.8704 75.8952)
-		(width 0.2)
+		(width 0.35)
 		(layer "F.Cu")
 		(net "/Signal_AMP")
@@
 		(start 151.7904 76.9112)
 		(end 154.171115 76.9112)
-		(width 0.2)
+		(width 0.35)
 		(layer "F.Cu")
 		(net "/Signal_AMP")
@@
 		(start 160.764448 75.8952)
 		(end 160.815248 75.946)
-		(width 0.2)
+		(width 0.35)
 		(layer "F.Cu")
 		(net "/Signal_AMP")
@@
 		(start 160.815248 75.946)
 		(end 161.668999 75.946)
-		(width 0.2)
+		(width 0.35)
 		(layer "F.Cu")
 		(net "/Signal_AMP")
@@
 		(start 151.3332 76.454)
 		(end 151.7904 76.9112)
-		(width 0.2)
+		(width 0.35)
 		(layer "F.Cu")
 		(net "/Signal_AMP")
@@
 		(start 152.950134 73.456)
 		(end 151.3332 75.072934)
-		(width 0.2)
+		(width 0.35)
 		(layer "F.Cu")
 		(net "/Signal_AMP")
@@
 		(start 154.190115 76.9302)
 		(end 155.8354 76.9302)
-		(width 0.2)
+		(width 0.35)
 		(layer "F.Cu")
 		(net "/Signal_AMP")
@@
 		(start 161.668999 75.946)
 		(end 162.0624 76.339401)
-		(width 0.2)
+		(width 0.35)
 		(layer "F.Cu")
 		(net "/Signal_AMP")
@@
 		(start 162.0624 76.339401)
 		(end 162.0624 77.1144)
-		(width 0.2)
+		(width 0.35)
 		(layer "F.Cu")
 		(net "/Signal_AMP")
@@
 		(start 154.171115 76.9112)
 		(end 154.190115 76.9302)
-		(width 0.2)
+		(width 0.35)
 		(layer "F.Cu")
 		(net "/Signal_AMP")
@@
 		(start 156.8704 75.8952)
 		(end 160.764448 75.8952)
-		(width 0.2)
+		(width 0.35)
 		(layer "F.Cu")
 		(net "/Signal_AMP")
@@
 	)
 	(segment
-		(start 159.7152 63.754)
-		(end 158.578349 62.617149)
+		(start 160.4772 64.516)
+		(end 160.4772 64.288825)
 		(width 0.2)
 		(layer "B.Cu")
@@
 	)
 	(segment
-		(start 158.578349 62.617149)
-		(end 158.578349 61.895)
+		(start 160.4772 64.288825)
+		(end 158.578349 62.389974)
 		(width 0.2)
 		(layer "B.Cu")
@@
 	)
 	(segment
-		(start 160.4772 64.516)
-		(end 159.7152 63.754)
+		(start 158.578349 62.389974)
+		(end 158.578349 61.895)
 		(width 0.2)
 		(layer "B.Cu")
@@
 	)
 	(segment
-		(start 165.000634 64.012)
-		(end 165.000634 65.2635)
-		(width 0.2)
-		(layer "F.Cu")
-		(net "/Vbias")
-	)
-	(segment
 		(start 163.9015 65.4605)
 		(end 165.027634 65.4605)
@@
 		(polygon
 			(pts
-				(xy 177.684193 66.94187) (xy 177.757849 66.875014) (xy 177.821639 66.830544) (xy 177.929436 66.786962)
-				(xy 177.999003 66.771897) (xy 178.104139 66.748317) (xy 178.240279 66.701659) (xy 178.109163 66.375478)
-				(xy 177.782982 66.244362) (xy 177.726686 66.419103) (xy 177.712743 66.485639) (xy 177.696254 66.560634)
-				(xy 177.670294 66.632395) (xy 177.623066 66.70948) (xy 177.542771 66.800448)
+				(xy 177.697997 66.928066) (xy 177.771653 66.86121) (xy 177.835443 66.81674) (xy 177.94324 66.773158)
+				(xy 178.012807 66.758093) (xy 178.117943 66.734513) (xy 178.254083 66.687855) (xy 178.122967 66.361674)
+				(xy 177.796786 66.230558) (xy 177.74049 66.405299) (xy 177.726547 66.471835) (xy 177.710058 66.54683)
+				(xy 177.684098 66.618591) (xy 177.63687 66.695676) (xy 177.556575 66.786644)
 			)
 		)
@@
 			)
 		)
-	)
-	(zone
-		(layers "F.Cu" "B.Cu" "B.SilkS")
-		(hatch edge 0.5)
-		(connect_pads
-			(clearance 0)
-		)
-		(min_thickness 0.25)
-		(keepout
-			(tracks allowed)
-			(vias allowed)
-			(pads allowed)
-			(copperpour not_allowed)
-			(footprints allowed)
-		)
-		(placement
-			(enabled no)
-			(sheetname "/")
-		)
-		(fill
-			(thermal_gap 0.5)
-			(thermal_bridge_width 0.5)
-			(island_removal_mode 0)
-		)
-		(polygon
-			(pts
-				(xy 108.92689 91.619072) (xy 116.665791 96.037237) (xy 113.89 100.1) (xy 105.234468 94.956259) (xy 105.234468 94.688709)
-			)
-		)
-	)
-	(zone
-		(net "GNDA")
-		(layer "B.Cu")
-		(hatch edge 0.5)
-		(priority 1)
-		(connect_pads
-			(clearance 0)
-		)
-		(min_thickness 0.25)
-		(fill yes
-			(thermal_gap 0.5)
-			(thermal_bridge_width 0.5)
-			(island_removal_mode 0)
-		)
-		(polygon
-			(pts
-				(xy 128.268643 90.716811) (xy 139.018643 95.716811) (xy 136.268643 98.466811) (xy 136.268643 101.966811)
-				(xy 122.018643 101.966811) (xy 122.018643 91.716811)
-			)
-		)

Commit message: Signed-off-by: lokimetasmith <lokimail@gmail.com>
Parts:
- moved NT5 0.58 mm to (163.1, 76.2)
- moved R8 0.16 mm to (164.9, 71.0)
Routing:
- net GNDA: track 5.93 -> 11.9 mm
- net VDDA: track 29.6 -> 29.7 mm, vias 3 -> 2
Changed lines of the file:
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@@
 	(footprint "NetTie:NetTie-2_SMD_Pad0.5mm"
 		(layer "F.Cu")
-		(at 163.0172 76.7588 -90)
+		(at 163.07 76.18 -90)
 		(descr "Net tie, 2 pin, 0.5mm square SMD pads")
 		(tags "net tie")
@@
 	(footprint "Resistor_SMD:R_0805_2012Metric"
 		(layer "F.Cu")
-		(at 165.000634 71.12)
+		(at 164.94 70.97)
 		(descr "Resistor SMD 0805 (2012 Metric), square (rectangular) end terminal, IPC-7351 nominal, (Body size source: IPC-SM-782 page 72, https://www.pcb-3d.com/wordpress/wp-content/uploads/ipc-sm-782a_amendment_1_and_2.pdf)")
 		(tags "resistor")
@@
 	)
 	(segment
+		(start 168.0624 77.1144)
+		(end 168.0624 75.8884)
+		(width 0.2)
+		(layer "F.Cu")
+		(net "GNDA")
+	)
+	(segment
+		(start 168.0624 75.8884)
+		(end 167.4088 75.2348)
+		(width 0.2)
+		(layer "F.Cu")
+		(net "GNDA")
+	)
+	(segment
 		(start 165.913134 73.152)
 		(end 167.032634 73.152)
@@
 	)
 	(segment
+		(start 164.9958 77.0478)
+		(end 165.0624 77.1144)
+		(width 0.2)
+		(layer "F.Cu")
+		(net "GNDA")
+	)
+	(segment
 		(start 152.5036 75.436)
 		(end 152.0444 75.8952)
@@
 	)
 	(segment
+		(start 167.4088 76.768)
+		(end 167.0624 77.1144)
+		(width 0.2)
+		(layer "F.Cu")
+		(net "GNDA")
+	)
+	(segment
 		(start 163.2712 69.67)
 		(end 163.2712 68.7832)
@@
 	)
 	(segment
+		(start 164.9958 75.3618)
+		(end 164.9958 77.0478)
+		(width 0.2)
+		(layer "F.Cu")
+		(net "GNDA")
+	)
+	(segment
+		(start 167.4088 75.2348)
+		(end 167.4088 76.768)
+		(width 0.2)
+		(layer "F.Cu")
+		(net "GNDA")
+	)
+	(segment
 		(start 152.992634 75.436)
 		(end 152.5036 75.436)
@@
 	)
 	(segment
-		(start 157.14569 67.5132)
-		(end 161.462634 67.5132)
+		(start 162.137766 75.379366)
+		(end 162.056 75.379366)
 		(width 0.2)
 		(layer "F.Cu")
@@
 	)
 	(segment
-		(start 161.3916 67.9176)
-		(end 161.3916 68.072)
+		(start 157.14569 67.5132)
+		(end 161.462634 67.5132)
 		(width 0.2)
 		(layer "F.Cu")
@@
 	)
 	(segment
-		(start 162.137766 75.379366)
-		(end 162.056 75.379366)
+		(start 161.3916 67.9176)
+		(end 161.3916 68.072)
 		(width 0.2)
 		(layer "F.Cu")
@@
 	)
 	(segment
-		(start 162.056 75.379366)
-		(end 161.987634 75.311)
+		(start 163.0192 64.8716)
+		(end 163.0192 65.396)
 		(width 0.2)
 		(layer "F.Cu")
@@
 	)
 	(segment
-		(start 163.0192 64.8716)
-		(end 163.0192 65.396)
+		(start 161.962234 75.3364)
+		(end 156.8196 75.3364)
 		(width 0.2)
 		(layer "F.Cu")
@@
 	)
 	(segment
-		(start 161.962234 75.3364)
-		(end 156.8196 75.3364)
+		(start 162.4384 75.68)
+		(end 162.137766 75.379366)
 		(width 0.2)
 		(layer "F.Cu")
@@
 	)
 	(segment
-		(start 163.0172 76.2588)
-		(end 162.137766 75.379366)
-		(width 0.2)
-		(layer "F.Cu")
-		(net "/Vbias")
-	)
-	(segment
 		(start 161.6872 68.3676)
 		(end 161.760524 68.3676)
@@
 	)
 	(segment
+		(start 162.056 75.379366)
+		(end 161.987634 75.311)
+		(width 0.2)
+		(layer "F.Cu")
+		(net "/Vbias")
+	)
+	(segment
+		(start 163.07 75.68)
+		(end 162.4384 75.68)
+		(width 0.2)
+		(layer "F.Cu")
+		(net "/Vbias")
+	)
+	(segment
 		(start 162.0116 69.256524)
 		(end 161.987634 69.28049)
@@
 	)
 	(segment
+		(start 164.443068 74.418532)
+		(end 164.1094 74.7522)
+		(width 0.2)
+		(layer "F.Cu")
+		(net "VDDA")
+	)
+	(segment
 		(start 156.837634 72.9234)
 		(end 155.962635 72.9234)
@@
 	)
 	(segment
-		(start 155.5496 74.5236)
-		(end 155.4988 74.5236)
+		(start 164.900634 73.836744)
+		(end 164.79 73.947378)
 		(width 0.2)
 		(layer "F.Cu")
@@
 	)
 	(segment
-		(start 172.037634 68.6105)
-		(end 171.737634 68.9105)
+		(start 155.5496 74.5236)
+		(end 155.4988 74.5236)
 		(width 0.2)
 		(layer "F.Cu")
@@
 	)
 	(segment
-		(start 172.037634 67.9105)
-		(end 172.037634 68.6105)
+		(start 164.900634 72.559366)
+		(end 164.900634 73.836744)
+		(width 0.2)
+		(layer "F.Cu")
+		(net "VDDA")
+	)
+	(segment
+		(start 169.48 72.12)
+		(end 165.41589 72.12)
+		(width 0.2)
+		(layer "F.Cu")
+		(net "VDDA")
+	)
+	(segment
+		(start 172.04 68.612866)
+		(end 172.04 69.56)
 		(width 0.2)
 		(layer "F.Cu")
@@
 	)
 	(segment
+		(start 165.41589 72.12)
+		(end 165.377945 72.082055)
+		(width 0.2)
+		(layer "F.Cu")
+		(net "VDDA")
+	)
+	(segment
 		(start 164.0624 74.7992)
 		(end 164.1094 74.7522)
@@
 		(net "VDDA")
 	)
-	(via
-		(at 155.4988 74.5236)
-		(size 0.6)
-		(drill 0.3)
-		(layers "F.Cu" "B.Cu")
+	(segment
+		(start 172.037634 67.9105)
+		(end 172.037634 68.6105)
+		(width 0.2)
+		(layer "F.Cu")
 		(net "VDDA")
 	)
-	(via
-		(at 171.737634 68.9105)
-		(size 0.6)
-		(drill 0.3)
-		(layers "F.Cu" "B.Cu")
+	(segment
+		(start 164.443068 74.366932)
+		(end 164.443068 74.418532)
+		(width 0.2)
+		(layer "F.Cu")
 		(net "VDDA")
 	)
-	(via
-		(at 164.1094 74.7522)
-		(size 0.6)
-		(drill 0.3)
-		(layers "F.Cu" "B.Cu")
+	(segment
+		(start 165.377945 72.082055)
+		(end 164.900634 72.559366)
+		(width 0.2)
+		(layer "F.Cu")
 		(net "VDDA")
 	)
 	(segment
-		(start 164.9984 75.6412)
-		(end 164.1094 74.7522)
+		(start 164.79 73.947378)
+		(end 164.79 74.02)
 		(width 0.2)
-		(layer "B.Cu")
+		(layer "F.Cu")
 		(net "VDDA")
 	)
 	(segment
-		(start 163.8808 74.5236)
-		(end 164.1094 74.7522)
+		(start 172.04 69.56)
+		(end 169.48 72.12)
 		(width 0.2)
-		(layer "B.Cu")
+		(layer "F.Cu")
 		(net "VDDA")
 	)
 	(segment
-		(start 171.737634 68.9105)
-		(end 171.737634 69.968766)
+		(start 172.037634 68.6105)
+		(end 172.04 68.612866)
 		(width 0.2)
-		(layer "B.Cu")
+		(layer "F.Cu")
 		(net "VDDA")
 	)
 	(segment
-		(start 166.0652 75.6412)
-		(end 164.9984 75.6412)
+		(start 164.79 74.02)
+		(end 164.443068 74.366932)
 		(width 0.2)
-		(layer "B.Cu")
+		(layer "F.Cu")
+		(net "VDDA")
+	)
+	(via
+		(at 155.4988 74.5236)
+		(size 0.6)
+		(drill 0.3)
+		(layers "F.Cu" "B.Cu")
+		(net "VDDA")
+	)
+	(via
+		(at 164.1094 74.7522)
+		(size 0.6)
+		(drill 0.3)
+		(layers "F.Cu" "B.Cu")
 		(net "VDDA")
 	)
 	(segment
-		(start 155.4988 74.5236)
-		(end 163.8808 74.5236)
+		(start 163.8808 74.5236)
+		(end 164.1094 74.7522)
 		(width 0.2)
 		(layer "B.Cu")
@@
 	)
 	(segment
-		(start 171.737634 69.968766)
-		(end 166.0652 75.6412)
+		(start 155.4988 74.5236)
+		(end 163.8808 74.5236)
 		(width 0.2)
 		(layer "B.Cu")
