File: Pump/MCU_STM32.kicad_sch (KiCad schematic)
At the start: 0 parts

Commit message: refactor: Rename Daemon Pore/Sentinel to MR1 across codebase
- Replaced "Daemon Pore", "Sentinel", and related variations with "MR1" in files.
- Renamed files matching "sentinel" or "daemon-pore" to "mr1".
- Ensured file references, includes, makefiles, and render scripts are correctly pointed to the new names.
- Retained case formatting consistency (`MR1` for PascalCase/UPPER_CASE/Prose, `mr1` for snake_case/filenames).

Co-authored-by: google-labs-jules[bot] <161369871+google-labs-jules[bot]@users.noreply.github.com>
Other:
- company: Daemon Pore Open Source Project -> MR1 Open Source Project
- title: Sentinel Pump Module - STM32 Control Processor -> MR1 Pump Module - STM32 Control Processor
Changed lines of the file:
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@@
 	(paper "A4")
 	(title_block
-		(title "Sentinel Pump Module - STM32 Control Processor")
+		(title "MR1 Pump Module - STM32 Control Processor")
 		(date "2026-09-30")
 		(rev "1.0")
-		(company "Daemon Pore Open Source Project")
+		(company "MR1 Open Source Project")
 		(comment 1 "STM32G431CBU6 32-bit ARM Cortex-M4 MCU @ 170 MHz")
 		(comment 2 "Hardware I2C buses for pressure transducers, USB-PD, and SBU link")
