File: Pump/Power_PD.kicad_sch (KiCad schematic)
At the start: 0 parts

Commit message: refactor: Rename Daemon Pore/Sentinel to MR1 across codebase
- Replaced "Daemon Pore", "Sentinel", and related variations with "MR1" in files.
- Renamed files matching "sentinel" or "daemon-pore" to "mr1".
- Ensured file references, includes, makefiles, and render scripts are correctly pointed to the new names.
- Retained case formatting consistency (`MR1` for PascalCase/UPPER_CASE/Prose, `mr1` for snake_case/filenames).

Co-authored-by: google-labs-jules[bot] <161369871+google-labs-jules[bot]@users.noreply.github.com>
Other:
- company: Daemon Pore Open Source Project -> MR1 Open Source Project
- title: Sentinel Pump Module - USB-PD Sink & Regulated Power Subsystem -> MR1 Pump Module - USB-PD Sink & Regulated Power Subsystem
Changed lines of the file:
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@@
 	(paper "A4")
 	(title_block
-		(title "Sentinel Pump Module - USB-PD Sink & Regulated Power Subsystem")
+		(title "MR1 Pump Module - USB-PD Sink & Regulated Power Subsystem")
 		(date "2026-09-30")
 		(rev "1.0")
-		(company "Daemon Pore Open Source Project")
+		(company "MR1 Open Source Project")
 		(comment 1 "STUSB4500 autonomous USB-PD Sink (negotiates 9V/12V/15V/20V)")
 		(comment 2 "Synchronous Buck Converter (36V/3A) stepping down to clean +5V")
