File: Pump/Pressure_Sensors.kicad_sch (KiCad schematic)
At the start: 0 parts

Commit message: refactor: Rename Daemon Pore/Sentinel to MR1 across codebase
- Replaced "Daemon Pore", "Sentinel", and related variations with "MR1" in files.
- Renamed files matching "sentinel" or "daemon-pore" to "mr1".
- Ensured file references, includes, makefiles, and render scripts are correctly pointed to the new names.
- Retained case formatting consistency (`MR1` for PascalCase/UPPER_CASE/Prose, `mr1` for snake_case/filenames).

Co-authored-by: google-labs-jules[bot] <161369871+google-labs-jules[bot]@users.noreply.github.com>
Other:
- company: Daemon Pore Open Source Project -> MR1 Open Source Project
- title: Sentinel Pump Module - Dual Fluidic Pressure Transducers -> MR1 Pump Module - Dual Fluidic Pressure Transducers
Changed lines of the file:
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@@
 	(paper "A4")
 	(title_block
-		(title "Sentinel Pump Module - Dual Fluidic Pressure Transducers")
+		(title "MR1 Pump Module - Dual Fluidic Pressure Transducers")
 		(date "2026-09-30")
 		(rev "1.0")
-		(company "Daemon Pore Open Source Project")
+		(company "MR1 Open Source Project")
 		(comment 1 "Honeywell TruStability / ABP2 Series Microfluidic Pressure Transducers")
 		(comment 2 "Precision 24-bit delta-sigma I2C digital pressure and temperature sensing")
