File: Pump/Pump.kicad_pcb (KiCad board)
At the start: 4 copper layers, 88 x 88 mm, 18 parts, among them J1_HOST USB_C_HOST, J2_MR1 USB_C_MR1_OUT, U10_SENS2 ABP2_005PG_TRANS, U1_MCU STM32G431CBU6, U2_PD STUSB4500, U3_BUCK TPS54302, U4_LDO LD39050_3V3, U6_MUX TS3USB221, U7_DRV1 DRV8837C, U8_DRV2 DRV8837C, U9_SENS1 ABP2_015PG_CIS

Commit message: refactor: Rename Daemon Pore/Sentinel to MR1 across codebase
- Replaced "Daemon Pore", "Sentinel", and related variations with "MR1" in files.
- Renamed files matching "sentinel" or "daemon-pore" to "mr1".
- Ensured file references, includes, makefiles, and render scripts are correctly pointed to the new names.
- Retained case formatting consistency (`MR1` for PascalCase/UPPER_CASE/Prose, `mr1` for snake_case/filenames).

Co-authored-by: google-labs-jules[bot] <161369871+google-labs-jules[bot]@users.noreply.github.com>
Other:
- board text added: "MR1 PROJECT"
- board text added: "MR1 PUMP & USB-PD HUB REV 1.0"
- board text removed: "DAEMON PORE PROJECT"
- board text removed: "SENTINEL PUMP & USB-PD HUB REV 1.0"
Changed lines of the file:
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@@
 	(gr_line (start 56.0 142.0) (end 56.0 58.0) (stroke (width 0.15)) (layer "Edge.Cuts"))
 	(gr_line (start 56.0 58.0) (end 58.0 56.0) (stroke (width 0.15)) (layer "Edge.Cuts"))
-	(gr_text "SENTINEL PUMP & USB-PD HUB REV 1.0" (at 100.0 60.0) (layer "F.SilkS") (effects (font (size 1.5 1.5) (thickness 0.25))))
-	(gr_text "DAEMON PORE PROJECT" (at 100.0 140.0) (layer "F.SilkS") (effects (font (size 1.2 1.2) (thickness 0.2))))
+	(gr_text "MR1 PUMP & USB-PD HUB REV 1.0" (at 100.0 60.0) (layer "F.SilkS") (effects (font (size 1.5 1.5) (thickness 0.25))))
+	(gr_text "MR1 PROJECT" (at 100.0 140.0) (layer "F.SilkS") (effects (font (size 1.2 1.2) (thickness 0.2))))
 	(gr_text "HOST USB-PD IN" (at 85.0 66.5) (layer "F.SilkS") (effects (font (size 1.0 1.0) (thickness 0.18))))
 	(gr_text "MR1 READER OUT" (at 115.0 66.5) (layer "F.SilkS") (effects (font (size 1.0 1.0) (thickness 0.18))))
