File: Pump/USB_Interconnect.kicad_sch (KiCad schematic)
At the start: 0 parts

Commit message: refactor: Rename Daemon Pore/Sentinel to MR1 across codebase
- Replaced "Daemon Pore", "Sentinel", and related variations with "MR1" in files.
- Renamed files matching "sentinel" or "daemon-pore" to "mr1".
- Ensured file references, includes, makefiles, and render scripts are correctly pointed to the new names.
- Retained case formatting consistency (`MR1` for PascalCase/UPPER_CASE/Prose, `mr1` for snake_case/filenames).

Co-authored-by: google-labs-jules[bot] <161369871+google-labs-jules[bot]@users.noreply.github.com>
Other:
- company: Daemon Pore Open Source Project -> MR1 Open Source Project
- title: Sentinel Pump Module - Dual USB-C Interconnect & High-Speed Pass-Through -> MR1 Pump Module - Dual USB-C Interconnect & High-Speed Pass-Through
Changed lines of the file:
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@@
 	(paper "A4")
 	(title_block
-		(title "Sentinel Pump Module - Dual USB-C Interconnect & High-Speed Pass-Through")
+		(title "MR1 Pump Module - Dual USB-C Interconnect & High-Speed Pass-Through")
 		(date "2026-09-30")
 		(rev "1.0")
-		(company "Daemon Pore Open Source Project")
+		(company "MR1 Open Source Project")
 		(comment 1 "Dual USB-C Receptacles aligned to Housing_Pump_Case cutouts (X = +/-15 mm)")
 		(comment 2 "J1_HOST: USB-PD Power Sink & Host Data Port")
