File: Pump/Pump.kicad_sch (KiCad schematic)
At the start: 25 parts, among them J1 USB_C_HOST, J2 USB_C_MR1_OUT, J3 PUMP1_MOTOR, J4 PUMP2_MOTOR, J5 SWD_DEBUG, U1 STM32G431CBU6, U10 ABP2_005PG_TRANS, U2 STUSB4500, U3 TPS54302, U4 LD39050_3V3, U5 TPS22916, U6 TS3USB221, U7 DRV8837C, U8 DRV8837C, U9 ABP2_015PG_CIS

Commit message: refactor: Rename Daemon Pore/Sentinel to MR1 across codebase
- Replaced "Daemon Pore", "Sentinel", and related variations with "MR1" in files.
- Renamed files matching "sentinel" or "daemon-pore" to "mr1".
- Ensured file references, includes, makefiles, and render scripts are correctly pointed to the new names.
- Retained case formatting consistency (`MR1` for PascalCase/UPPER_CASE/Prose, `mr1` for snake_case/filenames).

Co-authored-by: google-labs-jules[bot] <161369871+google-labs-jules[bot]@users.noreply.github.com>
Other:
- note added: "=== MR1 PERISTALTIC PUMP & USB-PD HUB ARCHITECTURE === 1. Dual USB-C Receptacles aligned to Housing_Pump_Case back-wall cutouts (X = +/-15 mm) 2. STUSB4500 USB-PD Sink negotiates high-power 9V/12V VBUS for peristaltic pump motors 3. High-efficiency synchronous buck converter outputs clean +5V power to MR1 Nanopore Reader 4. TI TS3USB221 USB 2.0 switch passes 100 kHz streaming data straight throug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"
- note removed: "=== SENTINEL PERISTALTIC PUMP & USB-PD HUB ARCHITECTURE === 1. Dual USB-C Receptacles aligned to Housing_Pump_Case back-wall cutouts (X = +/-15 mm) 2. STUSB4500 USB-PD Sink negotiates high-power 9V/12V VBUS for peristaltic pump motors 3. High-efficiency synchronous buck converter outputs clean +5V power to MR1 Nanopore Reader 4. TI TS3USB221 USB 2.0 switch passes 100 kHz streaming data straight t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"
- company: Daemon Pore Open Source Project -> MR1 Open Source Project
- title: Sentinel Nanopore Reader - Peristaltic Pump & USB-PD Power Hub -> MR1 Nanopore Reader - Peristaltic Pump & USB-PD Power Hub
Changed lines of the file:
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@@
 	(paper "A3")
 	(title_block
-		(title "Sentinel Nanopore Reader - Peristaltic Pump & USB-PD Power Hub")
+		(title "MR1 Nanopore Reader - Peristaltic Pump & USB-PD Power Hub")
 		(date "2026-09-30")
 		(rev "1.0")
-		(company "Daemon Pore Open Source Project")
+		(company "MR1 Open Source Project")
 		(comment 1 "Dual USB-C Interface (Host USB-PD Sink + Regulated Clean 5V Output to MR1)")
 		(comment 2 "STM32G431 Control Processor + Dual Honeywell TruStability Pressure Transducers")
@@
 		)
 	)
-	(text "=== SENTINEL PERISTALTIC PUMP & USB-PD HUB ARCHITECTURE ===\n1. Dual USB-C Receptacles aligned to Housing_Pump_Case back-wall cutouts (X = +/-15 mm)\n2. STUSB4500 USB-PD Sink negotiates high-power 9V/12V VBUS for peristaltic pump motors\n3. High-efficiency synchronous buck converter outputs clean +5V power to MR1 Nanopore Reader\n4. TI TS3USB221 USB 2.0 switch passes 100 kHz streaming data straight through to Host laptop\n5. USB-C SBU1/SBU2 lines provide bidirectional I2C control link with auto-polarity detection\n6. Dual Honeywell TruStability / ABP2 microfluidic pressure transducers monitor Cis and Trans lines\n7. Hardware emergency cutoff gate immediately shuts down pumps upon leak detection"
+	(text "=== MR1 PERISTALTIC PUMP & USB-PD HUB ARCHITECTURE ===\n1. Dual USB-C Receptacles aligned to Housing_Pump_Case back-wall cutouts (X = +/-15 mm)\n2. STUSB4500 USB-PD Sink negotiates high-power 9V/12V VBUS for peristaltic pump motors\n3. High-efficiency synchronous buck converter outputs clean +5V power to MR1 Nanopore Reader\n4. TI TS3USB221 USB 2.0 switch passes 100 kHz streaming data straight through to Host laptop\n5. USB-C SBU1/SBU2 lines provide bidirectional I2C control link with auto-polarity detection\n6. Dual Honeywell TruStability / ABP2 microfluidic pressure transducers monitor Cis and Trans lines\n7. Hardware emergency cutoff gate immediately shuts down pumps upon leak detection"
 		(at 30.0 180.0 0)
 		(effects (font (size 1.5 1.5)) (justify left))

Commit message: added opamp_signal_conditioning and more refined repo
Parts:
- C1, C2: LCSC (none) -> C15850
- C3: LCSC (none) -> C45783
- C4, C5: LCSC (none) -> C15255
- J1, J2: LCSC (none) -> C7095263
- J3, J4: LCSC (none) -> C158012
- J5: LCSC (none) -> C2337
- L1: LCSC (none) -> C87642
- R1: LCSC (none) -> C60491
- R2: LCSC (none) -> C25363
- R3, R4: LCSC (none) -> C25900
- U1: LCSC (none) -> C529356
- U10: LCSC (none) -> GZP6847D-C040KPP
- U2: LCSC (none) -> C2678061
- U3: LCSC (none) -> C9864
- U4: LCSC (none) -> C91206
- U5: LCSC (none) -> C131941
- U6: LCSC (none) -> C130085
- U7, U8: LCSC (none) -> C191000
- U9: LCSC (none) -> GZP6847D-C100KPP
Changed lines of the file:
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@@
 		(property "Value" "STM32G431CBU6" (at 100 102.54 0) (effects (font (size 1.27 1.27))))
 		(property "Footprint" "Package_DFN_QFN:QFN-48-1EP_7x7mm_P0.5mm_EP5.6x5.6mm" (at 100 105.08 0) (hide yes) (effects (font (size 1.27 1.27))))
+		(property "LCSC" "C529356" (at 100 105.08 0) (hide yes) (effects (font (size 1.27 1.27))))
 		(instances
 			(project "Pump"
@@
 		(property "Value" "STUSB4500" (at 100 102.54 0) (effects (font (size 1.27 1.27))))
 		(property "Footprint" "Package_DFN_QFN:QFN-24-1EP_4x4mm_P0.5mm_EP2.6x2.6mm" (at 100 105.08 0) (hide yes) (effects (font (size 1.27 1.27))))
+		(property "LCSC" "C2678061" (at 100 105.08 0) (hide yes) (effects (font (size 1.27 1.27))))
 		(instances
 			(project "Pump"
@@
 		(property "Value" "TPS54302" (at 100 102.54 0) (effects (font (size 1.27 1.27))))
 		(property "Footprint" "Package_SO:SOIC-8_3.9x4.9mm_P1.27mm" (at 100 105.08 0) (hide yes) (effects (font (size 1.27 1.27))))
+		(property "LCSC" "C9864" (at 100 105.08 0) (hide yes) (effects (font (size 1.27 1.27))))
 		(instances
 			(project "Pump"
@@
 		(property "Value" "LD39050_3V3" (at 100 102.54 0) (effects (font (size 1.27 1.27))))
 		(property "Footprint" "Package_TO_SOT_SMD:SOT-23-5" (at 100 105.08 0) (hide yes) (effects (font (size 1.27 1.27))))
+		(property "LCSC" "C91206" (at 100 105.08 0) (hide yes) (effects (font (size 1.27 1.27))))
 		(instances
 			(project "Pump"
@@
 		(property "Value" "TPS22916" (at 100 102.54 0) (effects (font (size 1.27 1.27))))
 		(property "Footprint" "Package_CSP:WLCSP-4_0.78x0.78mm_P0.4mm" (at 100 105.08 0) (hide yes) (effects (font (size 1.27 1.27))))
+		(property "LCSC" "C131941" (at 100 105.08 0) (hide yes) (effects (font (size 1.27 1.27))))
 		(instances
 			(project "Pump"
@@
 		(property "Value" "TS3USB221" (at 100 102.54 0) (effects (font (size 1.27 1.27))))
 		(property "Footprint" "Package_DFN_QFN:QFN-10_1.5x2mm_P0.4mm" (at 100 105.08 0) (hide yes) (effects (font (size 1.27 1.27))))
+		(property "LCSC" "C130085" (at 100 105.08 0) (hide yes) (effects (font (size 1.27 1.27))))
 		(instances
 			(project "Pump"
@@
 		(property "Value" "DRV8837C" (at 100 102.54 0) (effects (font (size 1.27 1.27))))
 		(property "Footprint" "Package_SON:WSON-8-1EP_2x2mm_P0.5mm_EP0.9x1.6mm" (at 100 105.08 0) (hide yes) (effects (font (size 1.27 1.27))))
+		(property "LCSC" "C191000" (at 100 105.08 0) (hide yes) (effects (font (size 1.27 1.27))))
 		(instances
 			(project "Pump"
@@
 		(property "Value" "DRV8837C" (at 100 102.54 0) (effects (font (size 1.27 1.27))))
 		(property "Footprint" "Package_SON:WSON-8-1EP_2x2mm_P0.5mm_EP0.9x1.6mm" (at 100 105.08 0) (hide yes) (effects (font (size 1.27 1.27))))
+		(property "LCSC" "C191000" (at 100 105.08 0) (hide yes) (effects (font (size 1.27 1.27))))
 		(instances
 			(project "Pump"
@@
 		(property "Value" "ABP2_015PG_CIS" (at 100 102.54 0) (effects (font (size 1.27 1.27))))
 		(property "Footprint" "Sensor_Pressure:Honeywell_ABP_SMD" (at 100 105.08 0) (hide yes) (effects (font (size 1.27 1.27))))
+		(property "LCSC" "GZP6847D-C100KPP" (at 100 105.08 0) (hide yes) (effects (font (size 1.27 1.27))))
 		(instances
 			(project "Pump"
@@
 		(property "Value" "ABP2_005PG_TRANS" (at 100 102.54 0) (effects (font (size 1.27 1.27))))
 		(property "Footprint" "Sensor_Pressure:Honeywell_ABP_SMD" (at 100 105.08 0) (hide yes) (effects (font (size 1.27 1.27))))
+		(property "LCSC" "GZP6847D-C040KPP" (at 100 105.08 0) (hide yes) (effects (font (size 1.27 1.27))))
 		(instances
 			(project "Pump"
@@
 		(property "Value" "USB_C_HOST" (at 100 102.54 0) (effects (font (size 1.27 1.27))))
 		(property "Footprint" "Connector_USB:USB_C_Receptacle_GCT_USB4085" (at 100 105.08 0) (hide yes) (effects (font (size 1.27 1.27))))
+		(property "LCSC" "C7095263" (at 100 105.08 0) (hide yes) (effects (font (size 1.27 1.27))))
 		(instances
 			(project "Pump"
@@
 		(property "Value" "USB_C_MR1_OUT" (at 100 102.54 0) (effects (font (size 1.27 1.27))))
 		(property "Footprint" "Connector_USB:USB_C_Receptacle_GCT_USB4085" (at 100 105.08 0) (hide yes) (effects (font (size 1.27 1.27))))
+		(property "LCSC" "C7095263" (at 100 105.08 0) (hide yes) (effects (font (size 1.27 1.27))))
 		(instances
 			(project "Pump"
@@
 		(property "Value" "PUMP1_MOTOR" (at 100 102.54 0) (effects (font (size 1.27 1.27))))
 		(property "Footprint" "Connector_JST:JST_XH_B2B-XH-A_1x02_P2.50mm_Vertical" (at 100 105.08 0) (hide yes) (effects (font (size 1.27 1.27))))
+		(property "LCSC" "C158012" (at 100 105.08 0) (hide yes) (effects (font (size 1.27 1.27))))
 		(instances
 			(project "Pump"
@@
 		(property "Value" "PUMP2_MOTOR" (at 100 102.54 0) (effects (font (size 1.27 1.27))))
 		(property "Footprint" "Connector_JST:JST_XH_B2B-XH-A_1x02_P2.50mm_Vertical" (at 100 105.08 0) (hide yes) (effects (font (size 1.27 1.27))))
+		(property "LCSC" "C158012" (at 100 105.08 0) (hide yes) (effects (font (size 1.27 1.27))))
 		(instances
 			(project "Pump"
@@
 		(property "Value" "SWD_DEBUG" (at 100 102.54 0) (effects (font (size 1.27 1.27))))
 		(property "Footprint" "Connector_PinHeader_2.54mm:PinHeader_1x04_P2.54mm_Vertical" (at 100 105.08 0) (hide yes) (effects (font (size 1.27 1.27))))
+		(property "LCSC" "C2337" (at 100 105.08 0) (hide yes) (effects (font (size 1.27 1.27))))
 		(instances
 			(project "Pump"
@@
 		(property "Value" "10uF" (at 100 102.54 0) (effects (font (size 1.27 1.27))))
 		(property "Footprint" "Capacitor_SMD:C_0805_2012Metric" (at 100 105.08 0) (hide yes) (effects (font (size 1.27 1.27))))
+		(property "LCSC" "C15850" (at 100 105.08 0) (hide yes) (effects (font (size 1.27 1.27))))
 		(instances
 			(project "Pump"
@@
 		(property "Value" "10uF" (at 100 102.54 0) (effects (font (size 1.27 1.27))))
 		(property "Footprint" "Capacitor_SMD:C_0805_2012Metric" (at 100 105.08 0) (hide yes) (effects (font (size 1.27 1.27))))
+		(property "LCSC" "C15850" (at 100 105.08 0) (hide yes) (effects (font (size 1.27 1.27))))
 		(instances
 			(project "Pump"
@@
 		(property "Value" "22uF" (at 100 102.54 0) (effects (font (size 1.27 1.27))))
 		(property "Footprint" "Capacitor_SMD:C_0805_2012Metric" (at 100 105.08 0) (hide yes) (effects (font (size 1.27 1.27))))
+		(property "LCSC" "C45783" (at 100 105.08 0) (hide yes) (effects (font (size 1.27 1.27))))
 		(instances
 			(project "Pump"
@@
 		(property "Value" "100nF" (at 100 102.54 0) (effects (font (size 1.27 1.27))))
 		(property "Footprint" "Capacitor_SMD:C_0402_1005Metric" (at 100 105.08 0) (hide yes) (effects (font (size 1.27 1.27))))
+		(property "LCSC" "C15255" (at 100 105.08 0) (hide yes) (effects (font (size 1.27 1.27))))
 		(instances
 			(project "Pump"
@@
 		(property "Value" "100nF" (at 100 102.54 0) (effects (font (size 1.27 1.27))))
 		(property "Footprint" "Capacitor_SMD:C_0402_1005Metric" (at 100 105.08 0) (hide yes) (effects (font (size 1.27 1.27))))
+		(property "LCSC" "C15255" (at 100 105.08 0) (hide yes) (effects (font (size 1.27 1.27))))
 		(instances
 			(project "Pump"
@@
 		(property "Value" "4.7uH" (at 100 102.54 0) (effects (font (size 1.27 1.27))))
 		(property "Footprint" "Inductor_SMD:L_Bourns_SRR4018" (at 100 105.08 0) (hide yes) (effects (font (size 1.27 1.27))))
+		(property "LCSC" "C87642" (at 100 105.08 0) (hide yes) (effects (font (size 1.27 1.27))))
 		(instances
 			(project "Pump"
@@
 		(property "Value" "100k" (at 100 102.54 0) (effects (font (size 1.27 1.27))))
 		(property "Footprint" "Resistor_SMD:R_0402_1005Metric" (at 100 105.08 0) (hide yes) (effects (font (size 1.27 1.27))))
+		(property "LCSC" "C60491" (at 100 105.08 0) (hide yes) (effects (font (size 1.27 1.27))))
 		(instances
 			(project "Pump"
@@
 		(property "Value" "32.4k" (at 100 102.54 0) (effects (font (size 1.27 1.27))))
 		(property "Footprint" "Resistor_SMD:R_0402_1005Metric" (at 100 105.08 0) (hide yes) (effects (font (size 1.27 1.27))))
+		(property "LCSC" "C25363" (at 100 105.08 0) (hide yes) (effects (font (size 1.27 1.27))))
 		(instances
 			(project "Pump"
@@
 		(property "Value" "4.7k" (at 100 102.54 0) (effects (font (size 1.27 1.27))))
 		(property "Footprint" "Resistor_SMD:R_0402_1005Metric" (at 100 105.08 0) (hide yes) (effects (font (size 1.27 1.27))))
+		(property "LCSC" "C25900" (at 100 105.08 0) (hide yes) (effects (font (size 1.27 1.27))))
 		(instances
 			(project "Pump"
@@
 		(property "Value" "4.7k" (at 100 102.54 0) (effects (font (size 1.27 1.27))))
 		(property "Footprint" "Resistor_SMD:R_0402_1005Metric" (at 100 105.08 0) (hide yes) (effects (font (size 1.27 1.27))))
-		(instances
-			(project "Pump"
+		(property "LCSC" "C25900" (at 100 105.08 0) (hide yes) (effects (font (size 1.27 1.27))))
+		(instances
+			(project "Pump"
